Commit message: quadruped

File: body.urdf (robot description, URDF)
Before this commit: robot robot, 3 links, 2 joints
Links:
- added link BackLowerLeg, mass 1; collision box size=0.2 0.2 1; visual box size=0.2 0.2 1
- added link FrontLowerLeg, mass 1; collision box size=0.2 0.2 1; visual box size=0.2 0.2 1
- added link LeftLeg, mass 1; collision box size=1 0.2 0.2; visual box size=1 0.2 0.2
- added link LeftLowerLeg, mass 1; collision box size=0.2 0.2 1; visual box size=0.2 0.2 1
- added link RightLeg, mass 1; collision box size=1 0.2 0.2; visual box size=1 0.2 0.2
- added link RightLowerLeg, mass 1; collision box size=0.2 0.2 1; visual box size=0.2 0.2 1
- link BackLeg: geometry collision box size=0.2 1 0.2; visual box size=0.2 1 0.2
- link FrontLeg: geometry collision box size=0.2 1 0.2; visual box size=0.2 1 0.2
Joints:
- added joint BackLeg_BackLowerLeg: type revolute, parent BackLeg, child BackLowerLeg, origin xyz=0 -1 0 rpy=0 0 0, axis 1 0 0, limit lower=-3.14159 upper=3.14159 effort=0.0 velocity=0.0
- added joint FrontLeg_FrontLowerLeg: type revolute, parent FrontLeg, child FrontLowerLeg, origin xyz=0 1 0 rpy=0 0 0, axis 1 0 0, limit lower=-3.14159 upper=3.14159 effort=0.0 velocity=0.0
- added joint LeftLeg_LeftLowerLeg: type revolute, parent LeftLeg, child LeftLowerLeg, origin xyz=-1 0 0 rpy=0 0 0, axis 0 1 0, limit lower=-3.14159 upper=3.14159 effort=0.0 velocity=0.0
- added joint RightLeg_RightLowerLeg: type revolute, parent RightLeg, child RightLowerLeg, origin xyz=1 0 0 rpy=0 0 0, axis 0 1 0, limit lower=-3.14159 upper=3.14159 effort=0.0 velocity=0.0
- added joint Torso_LeftLeg: type revolute, parent Torso, child LeftLeg, origin xyz=-0.5 0 1 rpy=0 0 0, axis 0 1 0, limit lower=-3.14159 upper=3.14159 effort=0.0 velocity=0.0
- added joint Torso_RightLeg: type revolute, parent Torso, child RightLeg, origin xyz=0.5 0 1 rpy=0 0 0, axis 0 1 0, limit lower=-3.14159 upper=3.14159 effort=0.0 velocity=0.0
- joint Torso_BackLeg: axis 0 1 0 -> 1 0 0; origin xyz=0.5 0 1 rpy=0 0 0 -> xyz=0 -0.5 1 rpy=0 0 0
- joint Torso_FrontLeg: axis 0 1 0 -> 1 0 0; origin xyz=-0.5 0 1 rpy=0 0 0 -> xyz=0 0.5 1 rpy=0 0 0

Commit message: O

File: body.urdf (robot description, URDF)
Before this commit: robot robot, 9 links, 8 joints
Links:
- removed link LeftLowerLeg
- added link BackLeg2, mass 1; collision box size=0.2 0.6 0.2; visual box size=0.2 0.6 0.2
- added link BackLowerLeg2, mass 1; collision box size=0.2 0.2 1; visual box size=0.2 0.2 1
- added link FrontLeg2, mass 1; collision box size=0.2 0.6 0.2; visual box size=0.2 0.6 0.2
- added link FrontLowerLeg2, mass 1; collision box size=0.2 0.2 1; visual box size=0.2 0.2 1
- added link LeftLeg2, mass 1; collision box size=0.6 0.2 0.2; visual box size=0.6 0.2 0.2
- added link LeftLowerLeg2, mass 1; collision box size=0.2 0.2 1; visual box size=0.2 0.2 1
- added link RightLeg2, mass 1; collision box size=0.6 0.2 0.2; visual box size=0.6 0.2 0.2
- added link Shell1, mass 1; collision box size=0.8 0.6 0.3; visual box size=0.8 0.6 0.3
- added link Shell2, mass 1; collision box size=0.5 0.4 0.15; visual box size=0.5 0.4 0.15
- link BackLeg: geometry collision box size=0.2 0.6 0.2; visual box size=0.2 0.6 0.2
- link FrontLeg: geometry collision box size=0.2 0.6 0.2; visual box size=0.2 0.6 0.2
- link LeftLeg: geometry collision box size=0.6 0.2 0.2; visual box size=0.6 0.2 0.2
- link RightLeg: geometry collision box size=0.6 0.2 0.2; visual box size=0.6 0.2 0.2
- link Torso: geometry collision box size=1 1 0.5; visual box size=1 1 0.5
Joints:
- removed joint LeftLeg_LeftLowerLeg
- added joint BackLeg2_BackLowerLeg2: type revolute, parent BackLeg2, child BackLowerLeg2, origin xyz=0 -0.6 0 rpy=0 0 0, axis 1 0 0, limit lower=-3.14159 upper=3.14159 effort=0.0 velocity=0.0
- added joint FrontLeg2_FrontLowerLeg2: type revolute, parent FrontLeg2, child FrontLowerLeg2, origin xyz=0 0.6 0 rpy=0 0 0, axis 1 0 0, limit lower=-3.14159 upper=3.14159 effort=0.0 velocity=0.0
- added joint LeftLeg2_LeftLowerLeg2: type revolute, parent LeftLeg2, child LeftLowerLeg2, origin xyz=-0.6 0 0 rpy=0 0 0, axis 0 1 0, limit lower=-3.14159 upper=3.14159 effort=0.0 velocity=0.0
- added joint Shell1_Shell2: type revolute, parent Shell1, child Shell2, origin xyz=0 0 0.01 rpy=0 0 0, axis 0 0 1, limit lower=-3.14159 upper=3.14159 effort=0.0 velocity=0.0
- added joint Torso_BackLeg2: type revolute, parent Torso, child BackLeg2, origin xyz=-0.4 -0.5 1 rpy=0 0 0, axis 1 0 0, limit lower=-3.14159 upper=3.14159 effort=0.0 velocity=0.0
- added joint Torso_FrontLeg2: type revolute, parent Torso, child FrontLeg2, origin xyz=-0.4 0.5 1 rpy=0 0 0, axis 1 0 0, limit lower=-3.14159 upper=3.14159 effort=0.0 velocity=0.0
- added joint Torso_LeftLeg2: type revolute, parent Torso, child LeftLeg2, origin xyz=-0.5 -0.4 1 rpy=0 0 0, axis 0 1 0, limit lower=-3.14159 upper=3.14159 effort=0.0 velocity=0.0
- added joint Torso_RightLeg2: type revolute, parent Torso, child RightLeg2, origin xyz=0.5 -0.4 1 rpy=0 0 0, axis 0 1 0, limit lower=-3.14159 upper=3.14159 effort=0.0 velocity=0.0
- added joint Torso_Shell1: type revolute, parent Torso, child Shell1, origin xyz=0 0 1.3 rpy=0 0 0, axis 0 0 1, limit lower=-3.14159 upper=3.14159 effort=0.0 velocity=0.0
- joint BackLeg_BackLowerLeg: origin xyz=0 -1 0 rpy=0 0 0 -> xyz=0 -0.6 0 rpy=0 0 0
- joint FrontLeg_FrontLowerLeg: origin xyz=0 1 0 rpy=0 0 0 -> xyz=0 0.6 0 rpy=0 0 0
- joint RightLeg_RightLowerLeg: origin xyz=1 0 0 rpy=0 0 0 -> xyz=0.6 0 0 rpy=0 0 0
- joint Torso_BackLeg: origin xyz=0 -0.5 1 rpy=0 0 0 -> xyz=0.4 -0.5 1 rpy=0 0 0
- joint Torso_FrontLeg: origin xyz=0 0.5 1 rpy=0 0 0 -> xyz=0.4 0.5 1 rpy=0 0 0
- joint Torso_LeftLeg: origin xyz=-0.5 0 1 rpy=0 0 0 -> xyz=-0.5 0.4 1 rpy=0 0 0
- joint Torso_RightLeg: origin xyz=0.5 0 1 rpy=0 0 0 -> xyz=0.5 0.4 1 rpy=0 0 0

Commit message: randomized links and sizes

File: body.urdf (robot description, URDF)
Before this commit: robot robot, 17 links, 16 joints
Links:
- removed link BackLeg
- removed link BackLeg2
- removed link BackLowerLeg
- removed link BackLowerLeg2
- removed link FrontLeg
- removed link FrontLeg2
- removed link FrontLowerLeg
- removed link FrontLowerLeg2
- removed link LeftLeg
- removed link LeftLeg2
- removed link LeftLowerLeg2
- removed link RightLeg
- removed link RightLeg2
- removed link RightLowerLeg
- removed link Shell1
- removed link Shell2
- removed link Torso
- added link Link0, mass 1; collision box size=1.4715157792527565 1.9788813407446726 1.996425470913247; visual box size=1.4715157792527565 1.9788813407446726 1.996425470913247
- added link Link1, mass 1; collision box size=1.971584311310142 1.4086852676023631 1.1177710132576761; visual box size=1.971584311310142 1.4086852676023631 1.1177710132576761
- added link Link2, mass 1; collision box size=1.8958659889752016 1.5926920968359985 1.3866218067548735; visual box size=1.8958659889752016 1.5926920968359985 1.3866218067548735
- added link Link3, mass 1; collision box size=1.6033320995981644 1.409218478860932 0.20865592520052545; visual box size=1.6033320995981644 1.409218478860932 0.20865592520052545
- added link Link4, mass 1; collision box size=0.7355327390561369 0.5885209559569995 1.4330125480148066; visual box size=0.7355327390561369 0.5885209559569995 1.4330125480148066
- added link Link5, mass 1; collision box size=0.44756282304699035 0.42655148513414953 1.0772799743732127; visual box size=0.44756282304699035 0.42655148513414953 1.0772799743732127
- added link Link6, mass 1; collision box size=1.4586299511490026 0.515291291096838 1.714421253376874; visual box size=1.4586299511490026 0.515291291096838 1.714421253376874
- added link Link7, mass 1; collision box size=0.30695459921355533 0.14577142099187743 0.9524309921365562; visual box size=0.30695459921355533 0.14577142099187743 0.9524309921365562
- added link Link8, mass 1; collision box size=0.33944666974631654 1.087887787123019 1.9518717023643566; visual box size=0.33944666974631654 1.087887787123019 1.9518717023643566
Joints:
- removed joint BackLeg2_BackLowerLeg2
- removed joint BackLeg_BackLowerLeg
- removed joint FrontLeg2_FrontLowerLeg2
- removed joint FrontLeg_FrontLowerLeg
- removed joint LeftLeg2_LeftLowerLeg2
- removed joint RightLeg_RightLowerLeg
- removed joint Shell1_Shell2
- removed joint Torso_BackLeg
- removed joint Torso_BackLeg2
- removed joint Torso_FrontLeg
- removed joint Torso_FrontLeg2
- removed joint Torso_LeftLeg
- removed joint Torso_LeftLeg2
- removed joint Torso_RightLeg
- removed joint Torso_RightLeg2
- removed joint Torso_Shell1
- added joint Link0_Link1: type revolute, parent Link0, child Link1, origin xyz=0 0.9894406703723363 0.9982127354566235 rpy=0 0 0, axis 1 0 0, limit lower=-3.14159 upper=3.14159 effort=0.0 velocity=0.0
- added joint Link1_Link2: type revolute, parent Link1, child Link2, origin xyz=0 1.4086852676023631 0 rpy=0 0 0, axis 1 0 0, limit lower=-3.14159 upper=3.14159 effort=0.0 velocity=0.0
- added joint Link2_Link3: type revolute, parent Link2, child Link3, origin xyz=0 1.5926920968359985 0 rpy=0 0 0, axis 1 0 0, limit lower=-3.14159 upper=3.14159 effort=0.0 velocity=0.0
- added joint Link3_Link4: type revolute, parent Link3, child Link4, origin xyz=0 1.409218478860932 0 rpy=0 0 0, axis 1 0 0, limit lower=-3.14159 upper=3.14159 effort=0.0 velocity=0.0
- added joint Link4_Link5: type revolute, parent Link4, child Link5, origin xyz=0 0.5885209559569995 0 rpy=0 0 0, axis 1 0 0, limit lower=-3.14159 upper=3.14159 effort=0.0 velocity=0.0
- added joint Link5_Link6: type revolute, parent Link5, child Link6, origin xyz=0 0.42655148513414953 0 rpy=0 0 0, axis 1 0 0, limit lower=-3.14159 upper=3.14159 effort=0.0 velocity=0.0
- added joint Link6_Link7: type revolute, parent Link6, child Link7, origin xyz=0 0.515291291096838 0 rpy=0 0 0, axis 1 0 0, limit lower=-3.14159 upper=3.14159 effort=0.0 velocity=0.0
- added joint Link7_Link8: type revolute, parent Link7, child Link8, origin xyz=0 0.14577142099187743 0 rpy=0 0 0, axis 1 0 0, limit lower=-3.14159 upper=3.14159 effort=0.0 velocity=0.0

Commit message: adding color :)

File: body.urdf (robot description, URDF)
Before this commit: robot robot, 9 links, 8 joints
Links:
- removed link Link3
- removed link Link4
- removed link Link5
- removed link Link6
- removed link Link7
- removed link Link8
- link Link0: geometry collision box size=1.3259072664850131 1.4401667332089771 0.45889648903762936; visual box size=1.3259072664850131 1.4401667332089771 0.45889648903762936
- link Link1: geometry collision box size=1.1535168223774919 1.4976950084760328 1.5102963574153438; visual box size=1.1535168223774919 1.4976950084760328 1.5102963574153438
- link Link2: geometry collision box size=1.7097878194598721 1.7777831293149111 0.23755482938485478; visual box size=1.7097878194598721 1.7777831293149111 0.23755482938485478
Joints:
- removed joint Link2_Link3
- removed joint Link3_Link4
- removed joint Link4_Link5
- removed joint Link5_Link6
- removed joint Link6_Link7
- removed joint Link7_Link8
- joint Link0_Link1: origin xyz=0 0.9894406703723363 0.9982127354566235 rpy=0 0 0 -> xyz=0 0.7200833666044886 0.7551481787076719 rpy=0 0 0
- joint Link1_Link2: origin xyz=0 1.4086852676023631 0 rpy=0 0 0 -> xyz=0 1.4976950084760328 0 rpy=0 0 0

Commit message: random sensors

File: body.urdf (robot description, URDF)
Before this commit: robot robot, 3 links, 2 joints
Links:
- added link Link3, mass 1; collision box size=0.5131241008410765 0.8330648851925534 0.6255441111830775; visual box size=0.5131241008410765 0.8330648851925534 0.6255441111830775
- link Link0: geometry collision box size=1.1792839786456542 1.185127331684563 1.0160736596931552; visual box size=1.1792839786456542 1.185127331684563 1.0160736596931552
- link Link1: geometry collision box size=1.3449288999417879 1.1702625733263212 1.3841151100871094; visual box size=1.3449288999417879 1.1702625733263212 1.3841151100871094
- link Link2: geometry collision box size=1.4861529134601295 1.3461600513900793 0.824936771914098; visual box size=1.4861529134601295 1.3461600513900793 0.824936771914098
Joints:
- added joint Link2_Link3: type revolute, parent Link2, child Link3, origin xyz=0 1.3461600513900793 0 rpy=0 0 0, axis 1 0 0, limit lower=-3.14159 upper=3.14159 effort=0.0 velocity=0.0
- joint Link0_Link1: origin xyz=0 0.7200833666044886 0.7551481787076719 rpy=0 0 0 -> xyz=0 0.5925636658422815 0.6920575550435547 rpy=0 0 0
- joint Link1_Link2: origin xyz=0 1.4976950084760328 0 rpy=0 0 0 -> xyz=0 1.1702625733263212 0 rpy=0 0 0

Commit message: cleanup

File: body.urdf (robot description, URDF)
Before this commit: robot robot, 4 links, 3 joints
Links:
- added link Link4, mass 1; collision box size=0.8565981231319862 0.7055349530561756 1.4883369909391977; visual box size=0.8565981231319862 0.7055349530561756 1.4883369909391977
- added link Link5, mass 1; collision box size=1.1499931422997518 0.9505414786383783 0.8970817372591193; visual box size=1.1499931422997518 0.9505414786383783 0.8970817372591193
- link Link0: geometry collision box size=1.0740809765214387 0.5176445839629321 0.5929018794361293; visual box size=1.0740809765214387 0.5176445839629321 0.5929018794361293
- link Link1: geometry collision box size=0.8561751692777628 0.9727197053836157 1.428887429728516; visual box size=0.8561751692777628 0.9727197053836157 1.428887429728516
- link Link2: geometry collision box size=0.7562465688166029 0.7799575412508237 1.4907470183325648; visual box size=0.7562465688166029 0.7799575412508237 1.4907470183325648
- link Link3: geometry collision box size=1.455075705955899 1.1032439472826299 1.021894133463233; visual box size=1.455075705955899 1.1032439472826299 1.021894133463233
Joints:
- added joint Link3_Link4: type revolute, parent Link3, child Link4, origin xyz=0 1.1032439472826299 0 rpy=0 0 0, axis 1 0 0, limit lower=-3.14159 upper=3.14159 effort=0.0 velocity=0.0
- added joint Link4_Link5: type revolute, parent Link4, child Link5, origin xyz=0 0.7055349530561756 0 rpy=0 0 0, axis 1 0 0, limit lower=-3.14159 upper=3.14159 effort=0.0 velocity=0.0
- joint Link0_Link1: origin xyz=0 0.5925636658422815 0.6920575550435547 rpy=0 0 0 -> xyz=0 0.25882229198146606 0.7453735091662824 rpy=0 0 0
- joint Link1_Link2: origin xyz=0 1.1702625733263212 0 rpy=0 0 0 -> xyz=0 0.9727197053836157 0 rpy=0 0 0
- joint Link2_Link3: origin xyz=0 1.3461600513900793 0 rpy=0 0 0 -> xyz=0 0.7799575412508237 0 rpy=0 0 0

Commit message: preliminary a7

File: body.urdf (robot description, URDF)
Before this commit: robot robot, 6 links, 5 joints
Links:
- removed link Link4
- removed link Link5
- added link Link1ZLink0, mass 1; collision box size=0.5150733647800367 0.5262079277879718 0.7499541984347997; visual box size=0.5150733647800367 0.5262079277879718 0.7499541984347997
- added link Link1ZLink1, mass 1; collision box size=0.8632163290576633 0.6861544022382255 0.8961669925665077; visual box size=0.8632163290576633 0.6861544022382255 0.8961669925665077
- added link Link2MinXLink0, mass 1; collision box size=0.9349456563111384 0.9265518399121044 0.6029080236172742; visual box size=0.9349456563111384 0.9265518399121044 0.6029080236172742
- added link Link2MinXLink1, mass 1; collision box size=0.7179676839611673 0.5382235011483864 0.7909246957363926; visual box size=0.7179676839611673 0.5382235011483864 0.7909246957363926
- added link Link2ZLink0, mass 1; collision box size=0.5847165058605076 0.9555377694363532 0.940799686346072; visual box size=0.5847165058605076 0.9555377694363532 0.940799686346072
- added link Link2ZLink1, mass 1; collision box size=0.5847165058605076 0.8118922531000464 0.9907046490280054; visual box size=0.5847165058605076 0.8118922531000464 0.9907046490280054
- added link Link3XLink0, mass 1; collision box size=0.8487625047078295 0.94107666857129 0.5582092423356468; visual box size=0.8487625047078295 0.94107666857129 0.5582092423356468
- added link Link3XLink1, mass 1; collision box size=0.6954387844197484 0.6961325133719949 0.6257769085597964; visual box size=0.6954387844197484 0.6961325133719949 0.6257769085597964
- added link Link3XLink2, mass 1; collision box size=0.8987262773760505 0.6961325133719949 0.7778897391089913; visual box size=0.8987262773760505 0.6961325133719949 0.7778897391089913
- added link Link3ZLink0, mass 1; collision box size=0.6566841706697271 0.94107666857129 0.9384146501010368; visual box size=0.6566841706697271 0.94107666857129 0.9384146501010368
- added link Link3ZLink1, mass 1; collision box size=0.787273845655317 0.6101616377697511 0.7809844852013658; visual box size=0.787273845655317 0.6101616377697511 0.7809844852013658
- added link Link3ZLink2, mass 1; collision box size=0.8160992451739246 0.6101616377697511 0.8994631998193948; visual box size=0.8160992451739246 0.6101616377697511 0.8994631998193948
- link Link0: geometry collision box size=1.0390857568365406 0.8674111753306251 1.3265096614239922; visual box size=1.0390857568365406 0.8674111753306251 1.3265096614239922
- link Link1: geometry collision box size=0.5150733647800367 0.5262079277879718 1.3064439099403742; visual box size=0.5150733647800367 0.5262079277879718 1.3064439099403742
- link Link2: geometry collision box size=0.6540192949684379 1.2320196116864905 1.4304778239208655; visual box size=0.6540192949684379 1.2320196116864905 1.4304778239208655
- link Link3: geometry collision box size=0.6566841706697271 0.94107666857129 0.6245224122635584; visual box size=0.6566841706697271 0.94107666857129 0.6245224122635584
Joints:
- removed joint Link3_Link4
- removed joint Link4_Link5
- added joint Link1ZLink0_Link1ZLink1: type revolute, parent Link1ZLink0, child Link1ZLink1, origin xyz=0 0 0.7499541984347997 rpy=0 0 0, axis 0 0 1, limit lower=-3.14159 upper=3.14159 effort=0.0 velocity=0.0
- added joint Link1_Link1ZLink0: type revolute, parent Link1, child Link1ZLink0, origin xyz=0.25753668239001837 0 [0.66325483 0.65322195 0.71523891 0.31226121 0.43591423] rpy=0 0 0, axis 0 0 1, limit lower=-3.14159 upper=3.14159 effort=0.0 velocity=0.0
- added joint Link2MinXLink0_Link2MinXLink1: type revolute, parent Link2MinXLink0, child Link2MinXLink1, origin xyz=-0.9349456563111384 0 0 rpy=0 0 0, axis 1 0 0, limit lower=-3.14159 upper=3.14159 effort=0.0 velocity=0.0
- added joint Link2ZLink0_Link2ZLink1: type revolute, parent Link2ZLink0, child Link2ZLink1, origin xyz=0 0 0.940799686346072 rpy=0 0 0, axis 0 0 1, limit lower=-3.14159 upper=3.14159 effort=0.0 velocity=0.0
- added joint Link2_Link2MinXLink0: type revolute, parent Link2, child Link2MinXLink0, origin xyz=-0.32700964748421896 0.6160098058432453 0 rpy=0 0 0, axis 1 0 0, limit lower=-3.14159 upper=3.14159 effort=0.0 velocity=0.0
- added joint Link2_Link2ZLink0: type revolute, parent Link2, child Link2ZLink0, origin xyz=0.32700964748421896 0 [0.66325483 0.65322195 0.71523891 0.31226121 0.43591423] rpy=0 0 0, axis 0 0 1, limit lower=-3.14159 upper=3.14159 effort=0.0 velocity=0.0
- added joint Link3XLink0_Link3XLink1: type revolute, parent Link3XLink0, child Link3XLink1, origin xyz=0.8487625047078295 0 0 rpy=0 0 0, axis 1 0 0, limit lower=-3.14159 upper=3.14159 effort=0.0 velocity=0.0
- added joint Link3XLink1_Link3XLink2: type revolute, parent Link3XLink1, child Link3XLink2, origin xyz=0.6954387844197484 0 0 rpy=0 0 0, axis 1 0 0, limit lower=-3.14159 upper=3.14159 effort=0.0 velocity=0.0
- added joint Link3ZLink0_Link3ZLink1: type revolute, parent Link3ZLink0, child Link3ZLink1, origin xyz=0 0 0.9384146501010368 rpy=0 0 0, axis 0 0 1, limit lower=-3.14159 upper=3.14159 effort=0.0 velocity=0.0
- added joint Link3ZLink1_Link3ZLink2: type revolute, parent Link3ZLink1, child Link3ZLink2, origin xyz=0 0 0.7809844852013658 rpy=0 0 0, axis 0 0 1, limit lower=-3.14159 upper=3.14159 effort=0.0 velocity=0.0
- added joint Link3_Link3XLink0: type revolute, parent Link3, child Link3XLink0, origin xyz=0.32834208533486353 0.470538334285645 0 rpy=0 0 0, axis 1 0 0, limit lower=-3.14159 upper=3.14159 effort=0.0 velocity=0.0
- added joint Link3_Link3ZLink0: type revolute, parent Link3, child Link3ZLink0, origin xyz=0.32834208533486353 0 [0.66325483 0.65322195 0.71523891 0.31226121 0.43591423] rpy=0 0 0, axis 0 0 1, limit lower=-3.14159 upper=3.14159 effort=0.0 velocity=0.0
- joint Link0_Link1: origin xyz=0 0.25882229198146606 0.7453735091662824 rpy=0 0 0 -> xyz=0 0.43370558766531253 0.7152389119604328 rpy=0 0 0
- joint Link1_Link2: origin xyz=0 0.9727197053836157 0 rpy=0 0 0 -> xyz=0 0.5262079277879718 0 rpy=0 0 0
- joint Link2_Link3: origin xyz=0 0.7799575412508237 0 rpy=0 0 0 -> xyz=0 1.2320196116864905 0 rpy=0 0 0
