Commit message: z blocks

File: body.urdf (robot description, URDF)
Before this commit: robot robot, 16 links, 15 joints
Links:
- removed link Link2MinXLink1
- removed link Link2ZLink1
- removed link Link3
- removed link Link3XLink0
- removed link Link3XLink1
- removed link Link3XLink2
- removed link Link3ZLink0
- removed link Link3ZLink1
- removed link Link3ZLink2
- added link Link1MinXLink0, mass 1; collision box size=0.8754907514201201 0.6607621314468723 0.6701365130175606; visual box size=0.8754907514201201 0.6607621314468723 0.6701365130175606
- added link Link1XLink0, mass 1; collision box size=0.8312389484466914 0.932690409145379 0.9163531184383933; visual box size=0.8312389484466914 0.932690409145379 0.9163531184383933
- added link Link1XLink1, mass 1; collision box size=0.5864608369232605 0.7278820922873643 0.5005452672932788; visual box size=0.5864608369232605 0.7278820922873643 0.5005452672932788
- added link Link1XLink2, mass 1; collision box size=0.5385109744368906 0.5772659925108901 0.5963085384938059; visual box size=0.5385109744368906 0.5772659925108901 0.5963085384938059
- added link Link1ZLink2, mass 1; collision box size=0.7652224747829305 0.9560983410009019 0.7436169890824504; visual box size=0.7652224747829305 0.9560983410009019 0.7436169890824504
- link Link0: geometry collision box size=0.5098220806231708 0.6606450928826676 0.6406045032396969; visual box size=0.5098220806231708 0.6606450928826676 0.6406045032396969
- link Link1: geometry collision box size=1.4773454643420134 0.932690409145379 0.7556806751893469; visual box size=1.4773454643420134 0.932690409145379 0.7556806751893469
- link Link1ZLink0: geometry collision box size=0.6555393778130034 0.656536778314618 0.7999997221610748; visual box size=0.6555393778130034 0.656536778314618 0.7999997221610748
- link Link1ZLink1: geometry collision box size=0.6555393778130034 0.656536778314618 0.6179050551426521; visual box size=0.6555393778130034 0.656536778314618 0.6179050551426521
- link Link2: geometry collision box size=0.7158625755319169 1.3322397395912389 0.8396240490333694; visual box size=0.7158625755319169 1.3322397395912389 0.8396240490333694
- link Link2MinXLink0: geometry collision box size=0.8538762962208117 0.5205791981096685 0.6807283860842037; visual box size=0.8538762962208117 0.5205791981096685 0.6807283860842037
- link Link2ZLink0: geometry collision box size=0.6570429975850449 0.7076047645473459 0.8660754325897035; visual box size=0.6570429975850449 0.7076047645473459 0.8660754325897035
Joints:
- removed joint Link2MinXLink0_Link2MinXLink1
- removed joint Link2ZLink0_Link2ZLink1
- removed joint Link2_Link3
- removed joint Link3XLink0_Link3XLink1
- removed joint Link3XLink1_Link3XLink2
- removed joint Link3ZLink0_Link3ZLink1
- removed joint Link3ZLink1_Link3ZLink2
- removed joint Link3_Link3XLink0
- removed joint Link3_Link3ZLink0
- added joint Link1XLink0_Link1XLink1: type revolute, parent Link1XLink0, child Link1XLink1, origin xyz=0.8312389484466914 0 0 rpy=0 0 0, axis 1 0 0, limit lower=-3.14159 upper=3.14159 effort=0.0 velocity=0.0
- added joint Link1XLink1_Link1XLink2: type revolute, parent Link1XLink1, child Link1XLink2, origin xyz=0.5864608369232605 0 0 rpy=0 0 0, axis 1 0 0, limit lower=-3.14159 upper=3.14159 effort=0.0 velocity=0.0
- added joint Link1ZLink1_Link1ZLink2: type revolute, parent Link1ZLink1, child Link1ZLink2, origin xyz=0 0 0.6179050551426521 rpy=0 0 0, axis 0 0 1, limit lower=-3.14159 upper=3.14159 effort=0.0 velocity=0.0
- added joint Link1_Link1MinXLink0: type revolute, parent Link1, child Link1MinXLink0, origin xyz=-0.7386727321710067 0.4663452045726895 0 rpy=0 0 0, axis 1 0 0, limit lower=-3.14159 upper=3.14159 effort=0.0 velocity=0.0
- added joint Link1_Link1XLink0: type revolute, parent Link1, child Link1XLink0, origin xyz=0.7386727321710067 0.4663452045726895 0 rpy=0 0 0, axis 1 0 0, limit lower=-3.14159 upper=3.14159 effort=0.0 velocity=0.0
- joint Link0_Link1: origin xyz=0 0.43370558766531253 0.7152389119604328 rpy=0 0 0 -> xyz=0 0.3303225464413338 0.6518926456867749 rpy=0 0 0
- joint Link1ZLink0_Link1ZLink1: origin xyz=0 0 0.7499541984347997 rpy=0 0 0 -> xyz=0 0 0.7999997221610748 rpy=0 0 0
- joint Link1_Link1ZLink0: origin xyz=0.25753668239001837 0 [0.66325483 0.65322195 0.71523891 0.31226121 0.43591423] rpy=0 0 0 -> xyz=0 -0.4663452045726895 [1.92181351 2.26704203 2.51887215 3.91135587] rpy=0 0 0
- joint Link1_Link2: origin xyz=0 0.5262079277879718 0 rpy=0 0 0 -> xyz=0 0.932690409145379 0 rpy=0 0 0
- joint Link2_Link2MinXLink0: origin xyz=-0.32700964748421896 0.6160098058432453 0 rpy=0 0 0 -> xyz=-0.35793128776595845 0.6661198697956194 0 rpy=0 0 0
- joint Link2_Link2ZLink0: origin xyz=0.32700964748421896 0 [0.66325483 0.65322195 0.71523891 0.31226121 0.43591423] rpy=0 0 0 -> xyz=0 -0.6661198697956194 [1.92181351 2.26704203 2.51887215 3.91135587] rpy=0 0 0

Commit message: typos

File: body.urdf (robot description, URDF)
Before this commit: robot robot, 12 links, 11 joints
Links:
- removed link Link1XLink2
- removed link Link1ZLink0
- removed link Link1ZLink1
- removed link Link1ZLink2
- removed link Link2ZLink0
- added link Link2MinXLink1, mass 1; collision box size=0.6262150640538608 0.7157798628848435 0.8579986701072795; visual box size=0.6262150640538608 0.7157798628848435 0.8579986701072795
- added link Link2XLink0, mass 1; collision box size=0.7171562458420311 0.5422854381826757 0.6895093621048181; visual box size=0.7171562458420311 0.5422854381826757 0.6895093621048181
- added link Link2XLink1, mass 1; collision box size=0.8944189943022071 0.5422854381826757 0.5995129051631742; visual box size=0.8944189943022071 0.5422854381826757 0.5995129051631742
- added link Link3, mass 1; collision box size=1.0320161247331305 1.3353606986513191 1.387141470699401; visual box size=1.0320161247331305 1.3353606986513191 1.387141470699401
- added link Link3ZLink0, mass 1; collision box size=0.6524430383589659 0.7270471917237309 0.897205072083166; visual box size=0.6524430383589659 0.7270471917237309 0.897205072083166
- added link Link3ZLink1, mass 1; collision box size=0.6524430383589659 0.7270471917237309 0.7963694517044902; visual box size=0.6524430383589659 0.7270471917237309 0.7963694517044902
- added link Link4, mass 1; collision box size=0.8670112081721517 1.2970986551051775 0.55566738991666; visual box size=0.8670112081721517 1.2970986551051775 0.55566738991666
- added link Link4MinXLink0, mass 1; collision box size=0.7335083566699794 0.8583222372573466 0.5220038559322748; visual box size=0.7335083566699794 0.8583222372573466 0.5220038559322748
- added link Link4ZLink0, mass 1; collision box size=0.8339361837889834 0.6718056439899275 0.8358376872678976; visual box size=0.8339361837889834 0.6718056439899275 0.8358376872678976
- added link Link5, mass 1; collision box size=0.8922683113798471 1.268876099800507 1.1696866004039657; visual box size=0.8922683113798471 1.268876099800507 1.1696866004039657
- added link Link5XLink0, mass 1; collision box size=0.9228766742435077 0.7564156550566363 0.6969360756817713; visual box size=0.9228766742435077 0.7564156550566363 0.6969360756817713
- link Link0: geometry collision box size=0.9644827517089818 1.1777912513116258 0.9718708853200249; visual box size=0.9644827517089818 1.1777912513116258 0.9718708853200249
- link Link1: geometry collision box size=0.6273061216090596 0.975234959034219 1.239500899334318; visual box size=0.6273061216090596 0.975234959034219 1.239500899334318
- link Link1MinXLink0: geometry collision box size=0.9460269023980526 0.7071994623068861 0.9782335112403986; visual box size=0.9460269023980526 0.7071994623068861 0.9782335112403986
- link Link1XLink0: geometry collision box size=0.7108142506169426 0.9596756613764718 0.6882038195328867; visual box size=0.7108142506169426 0.9596756613764718 0.6882038195328867
- link Link1XLink1: geometry collision box size=0.8832990986685153 0.5201324526507564 0.8271881622238841; visual box size=0.8832990986685153 0.5201324526507564 0.8271881622238841
- link Link2: geometry collision box size=1.1320259634820662 0.9007298271806301 1.2802639315242665; visual box size=1.1320259634820662 0.9007298271806301 1.2802639315242665
- link Link2MinXLink0: geometry collision box size=0.5069707123335523 0.7157798628848435 0.8114899173123588; visual box size=0.5069707123335523 0.7157798628848435 0.8114899173123588
Joints:
- removed joint Link1XLink1_Link1XLink2
- removed joint Link1ZLink0_Link1ZLink1
- removed joint Link1ZLink1_Link1ZLink2
- removed joint Link1_Link1ZLink0
- removed joint Link2_Link2ZLink0
- added joint Link2MinXLink0_Link2MinXLink1: type revolute, parent Link2MinXLink0, child Link2MinXLink1, origin xyz=-0.5069707123335523 0 0 rpy=0 0 0, axis 1 0 0, limit lower=-3.14159 upper=3.14159 effort=0.0 velocity=0.0
- added joint Link2XLink0_Link2XLink1: type revolute, parent Link2XLink0, child Link2XLink1, origin xyz=0.7171562458420311 0 0 rpy=0 0 0, axis 1 0 0, limit lower=-3.14159 upper=3.14159 effort=0.0 velocity=0.0
- added joint Link2_Link2XLink0: type revolute, parent Link2, child Link2XLink0, origin xyz=0.5660129817410331 0.45036491359031505 0 rpy=0 0 0, axis 1 0 0, limit lower=-3.14159 upper=3.14159 effort=0.0 velocity=0.0
- added joint Link2_Link3: type revolute, parent Link2, child Link3, origin xyz=0 0.9007298271806301 0 rpy=0 0 0, axis 1 0 0, limit lower=-3.14159 upper=3.14159 effort=0.0 velocity=0.0
- added joint Link3ZLink0_Link3ZLink1: type revolute, parent Link3ZLink0, child Link3ZLink1, origin xyz=0 0 0.897205072083166 rpy=0 0 0, axis 0 0 1, limit lower=-3.14159 upper=3.14159 effort=0.0 velocity=0.0
- added joint Link3_Link3ZLink0: type revolute, parent Link3, child Link3ZLink0, origin xyz=0 -0.6676803493256596 [2.91561266 3.7185027  3.84079179 4.16142441 1.66700217 3.5090598  4.4527399 ] rpy=0 0 0, axis 0 0 1, limit lower=-3.14159 upper=3.14159 effort=0.0 velocity=0.0
- added joint Link3_Link4: type revolute, parent Link3, child Link4, origin xyz=0 1.3353606986513191 0 rpy=0 0 0, axis 1 0 0, limit lower=-3.14159 upper=3.14159 effort=0.0 velocity=0.0
- added joint Link4_Link4MinXLink0: type revolute, parent Link4, child Link4MinXLink0, origin xyz=-0.43350560408607586 0.6485493275525888 0 rpy=0 0 0, axis 1 0 0, limit lower=-3.14159 upper=3.14159 effort=0.0 velocity=0.0
- added joint Link4_Link4ZLink0: type revolute, parent Link4, child Link4ZLink0, origin xyz=0 -0.6485493275525888 [2.91561266 3.7185027  3.84079179 4.16142441 1.66700217 3.5090598  4.4527399 ] rpy=0 0 0, axis 0 0 1, limit lower=-3.14159 upper=3.14159 effort=0.0 velocity=0.0
- added joint Link4_Link5: type revolute, parent Link4, child Link5, origin xyz=0 1.2970986551051775 0 rpy=0 0 0, axis 1 0 0, limit lower=-3.14159 upper=3.14159 effort=0.0 velocity=0.0
- added joint Link5_Link5XLink0: type revolute, parent Link5, child Link5XLink0, origin xyz=0.44613415568992354 0.6344380499002535 0 rpy=0 0 0, axis 1 0 0, limit lower=-3.14159 upper=3.14159 effort=0.0 velocity=0.0
- joint Link0_Link1: origin xyz=0 0.3303225464413338 0.6518926456867749 rpy=0 0 0 -> xyz=0 0.5888956256558129 0.7421233171234125 rpy=0 0 0
- joint Link1XLink0_Link1XLink1: origin xyz=0.8312389484466914 0 0 rpy=0 0 0 -> xyz=0.7108142506169426 0 0 rpy=0 0 0
- joint Link1_Link1MinXLink0: origin xyz=-0.7386727321710067 0.4663452045726895 0 rpy=0 0 0 -> xyz=-0.3136530608045298 0.4876174795171095 0 rpy=0 0 0
- joint Link1_Link1XLink0: origin xyz=0.7386727321710067 0.4663452045726895 0 rpy=0 0 0 -> xyz=0.3136530608045298 0.4876174795171095 0 rpy=0 0 0
- joint Link1_Link2: origin xyz=0 0.932690409145379 0 rpy=0 0 0 -> xyz=0 0.975234959034219 0 rpy=0 0 0
- joint Link2_Link2MinXLink0: origin xyz=-0.35793128776595845 0.6661198697956194 0 rpy=0 0 0 -> xyz=-0.5660129817410331 0.45036491359031505 0 rpy=0 0 0

Commit message: edit

File: body.urdf (robot description, URDF)
Before this commit: robot robot, 18 links, 17 joints
Links:
- removed link Link1MinXLink0
- removed link Link2MinXLink1
- removed link Link2XLink1
- removed link Link3ZLink1
- removed link Link4
- removed link Link4MinXLink0
- removed link Link4ZLink0
- removed link Link5
- removed link Link5XLink0
- added link Link2ZLink0, mass 1; collision box size=0.5864359265532006 0.9281264177642923 0.6253902401885905; visual box size=0.5864359265532006 0.9281264177642923 0.6253902401885905
- added link Link3MinXLink0, mass 1; collision box size=0.9637145854184892 0.7184828926514617 0.7530296942565208; visual box size=0.9637145854184892 0.7184828926514617 0.7530296942565208
- added link Link3MinXLink1, mass 1; collision box size=0.8029472144879135 0.7184828926514617 0.9614213861105816; visual box size=0.8029472144879135 0.7184828926514617 0.9614213861105816
- added link Link3XLink0, mass 1; collision box size=0.8896386929508217 0.7364988210815241 0.7580706736769504; visual box size=0.8896386929508217 0.7364988210815241 0.7580706736769504
- added link Link3XLink1, mass 1; collision box size=0.8832237681382225 0.7364988210815241 0.8480878485841941; visual box size=0.8832237681382225 0.7364988210815241 0.8480878485841941
- link Link0: geometry collision box size=0.695961891076385 0.6158352789671936 0.7499251940158412; visual box size=0.695961891076385 0.6158352789671936 0.7499251940158412
- link Link1: geometry collision box size=0.870908524155756 1.3482248600712223 0.7712005799898127; visual box size=0.870908524155756 1.3482248600712223 0.7712005799898127
- link Link1XLink0: geometry collision box size=0.8246317092591938 0.6285525964337848 0.7521183974233039; visual box size=0.8246317092591938 0.6285525964337848 0.7521183974233039
- link Link1XLink1: geometry collision box size=0.8300085786461922 0.6285525964337848 0.5148562954266425; visual box size=0.8300085786461922 0.6285525964337848 0.5148562954266425
- link Link2: geometry collision box size=0.5864359265532006 1.167557536979364 1.1205575616726962; visual box size=0.5864359265532006 1.167557536979364 1.1205575616726962
- link Link2MinXLink0: geometry collision box size=0.6023824260214328 0.55447937714717 0.8688829961681155; visual box size=0.6023824260214328 0.55447937714717 0.8688829961681155
- link Link2XLink0: geometry collision box size=0.626043450372916 0.6295596437038427 0.7511387365955885; visual box size=0.626043450372916 0.6295596437038427 0.7511387365955885
- link Link3: geometry collision box size=1.0464378094432492 1.3157467499064193 1.0109638657664934; visual box size=1.0464378094432492 1.3157467499064193 1.0109638657664934
- link Link3ZLink0: geometry collision box size=0.7778090307968426 0.8532021918240775 0.8031851619218164; visual box size=0.7778090307968426 0.8532021918240775 0.8031851619218164
Joints:
- removed joint Link1_Link1MinXLink0
- removed joint Link2MinXLink0_Link2MinXLink1
- removed joint Link2XLink0_Link2XLink1
- removed joint Link3ZLink0_Link3ZLink1
- removed joint Link3_Link4
- removed joint Link4_Link4MinXLink0
- removed joint Link4_Link4ZLink0
- removed joint Link4_Link5
- removed joint Link5_Link5XLink0
- added joint Link2_Link2ZLink0: type revolute, parent Link2, child Link2ZLink0, origin xyz=0 -0.583778768489682 [0.3749626  0.38560029 0.56027878 0.50548193 0.35031212] rpy=0 0 0, axis 0 0 1, limit lower=-3.14159 upper=3.14159 effort=0.0 velocity=0.0
- added joint Link3MinXLink0_Link3MinXLink1: type revolute, parent Link3MinXLink0, child Link3MinXLink1, origin xyz=-0.9637145854184892 0 0 rpy=0 0 0, axis 1 0 0, limit lower=-3.14159 upper=3.14159 effort=0.0 velocity=0.0
- added joint Link3XLink0_Link3XLink1: type revolute, parent Link3XLink0, child Link3XLink1, origin xyz=0.8896386929508217 0 0 rpy=0 0 0, axis 1 0 0, limit lower=-3.14159 upper=3.14159 effort=0.0 velocity=0.0
- added joint Link3_Link3MinXLink0: type revolute, parent Link3, child Link3MinXLink0, origin xyz=-0.5232189047216246 0.6578733749532096 0 rpy=0 0 0, axis 1 0 0, limit lower=-3.14159 upper=3.14159 effort=0.0 velocity=0.0
- added joint Link3_Link3XLink0: type revolute, parent Link3, child Link3XLink0, origin xyz=0.5232189047216246 0.6578733749532096 0 rpy=0 0 0, axis 1 0 0, limit lower=-3.14159 upper=3.14159 effort=0.0 velocity=0.0
- joint Link0_Link1: origin xyz=0 0.5888956256558129 0.7421233171234125 rpy=0 0 0 -> xyz=0 0.3079176394835968 0.5602787808363481 rpy=0 0 0
- joint Link1XLink0_Link1XLink1: origin xyz=0.7108142506169426 0 0 rpy=0 0 0 -> xyz=0.8246317092591938 0 0 rpy=0 0 0
- joint Link1_Link1XLink0: origin xyz=0.3136530608045298 0.4876174795171095 0 rpy=0 0 0 -> xyz=0.435454262077878 0.6741124300356112 0 rpy=0 0 0
- joint Link1_Link2: origin xyz=0 0.975234959034219 0 rpy=0 0 0 -> xyz=0 1.3482248600712223 0 rpy=0 0 0
- joint Link2_Link2MinXLink0: origin xyz=-0.5660129817410331 0.45036491359031505 0 rpy=0 0 0 -> xyz=-0.2932179632766003 0.583778768489682 0 rpy=0 0 0
- joint Link2_Link2XLink0: origin xyz=0.5660129817410331 0.45036491359031505 0 rpy=0 0 0 -> xyz=0.2932179632766003 0.583778768489682 0 rpy=0 0 0
- joint Link2_Link3: origin xyz=0 0.9007298271806301 0 rpy=0 0 0 -> xyz=0 1.167557536979364 0 rpy=0 0 0
- joint Link3_Link3ZLink0: origin xyz=0 -0.6676803493256596 [2.91561266 3.7185027  3.84079179 4.16142441 1.66700217 3.5090598  4.4527399 ] rpy=0 0 0 -> xyz=0 -0.6578733749532096 [0.3749626  0.38560029 0.56027878 0.50548193 0.35031212] rpy=0 0 0
