Commit message: updates

File: body.urdf (robot description, URDF)
Before this commit: robot robot, 14 links, 13 joints
Links:
- removed link Link1XLink1
- removed link Link2ZLink0
- added link Link1ZLink0, mass 1; collision box size=0.8247768043628712 0.5317324262196261 0.5512775077162138; visual box size=0.8247768043628712 0.5317324262196261 0.5512775077162138
- added link Link3XLink2, mass 1; collision box size=0.9742038978868903 0.5458716264817558 0.5700688060198874; visual box size=0.9742038978868903 0.5458716264817558 0.5700688060198874
- added link Link3ZLink1, mass 1; collision box size=0.9432582294312156 0.7472784743989974 0.9500488591895191; visual box size=0.9432582294312156 0.7472784743989974 0.9500488591895191
- added link Link4, mass 1; collision box size=0.8044207059996972 0.5724500855735579 1.0369027695656712; visual box size=0.8044207059996972 0.5724500855735579 1.0369027695656712
- added link Link4MinXLink0, mass 1; collision box size=0.5702196198438354 0.5724500855735579 0.7882207813729096; visual box size=0.5702196198438354 0.5724500855735579 0.7882207813729096
- added link Link4MinXLink1, mass 1; collision box size=0.8170859822595409 0.6340604150859717 0.6467978058543227; visual box size=0.8170859822595409 0.6340604150859717 0.6467978058543227
- added link Link4XLink0, mass 1; collision box size=0.6161413023397249 0.535755085958094 0.7586855932602034; visual box size=0.6161413023397249 0.535755085958094 0.7586855932602034
- added link Link4ZLink0, mass 1; collision box size=0.6669519014242027 0.5724500855735579 0.6905325550903523; visual box size=0.6669519014242027 0.5724500855735579 0.6905325550903523
- added link Link5, mass 1; collision box size=1.2203225708195409 0.9724794492916892 0.7393264118363885; visual box size=1.2203225708195409 0.9724794492916892 0.7393264118363885
- added link Link5MinXLink0, mass 1; collision box size=0.6997286672416282 0.6579749541542452 0.9488036044681691; visual box size=0.6997286672416282 0.6579749541542452 0.9488036044681691
- added link Link5XLink0, mass 1; collision box size=0.8608852501876022 0.5767750769778129 0.7826821473342618; visual box size=0.8608852501876022 0.5767750769778129 0.7826821473342618
- added link Link5ZLink0, mass 1; collision box size=0.7544410242996213 0.914638185002552 0.7351916746220126; visual box size=0.7544410242996213 0.914638185002552 0.7351916746220126
- link Link0: geometry collision box size=0.7319036431060393 0.6133605015786847 1.139761121095375; visual box size=0.7319036431060393 0.6133605015786847 1.139761121095375
- link Link1: geometry collision box size=0.8247768043628712 0.5317324262196261 1.3626753350157763; visual box size=0.8247768043628712 0.5317324262196261 1.3626753350157763
- link Link1XLink0: geometry collision box size=0.9256896730604203 0.5317324262196261 0.9930063773085074; visual box size=0.9256896730604203 0.5317324262196261 0.9930063773085074
- link Link2: geometry collision box size=0.8285636544242897 0.6464129644811623 0.8021154688836524; visual box size=0.8285636544242897 0.6464129644811623 0.8021154688836524
- link Link2MinXLink0: geometry collision box size=0.6631753978379646 0.5114330167748792 0.779141133863006; visual box size=0.6631753978379646 0.5114330167748792 0.779141133863006
- link Link2XLink0: geometry collision box size=0.6960643291512534 0.6464129644811623 0.5066951223386589; visual box size=0.6960643291512534 0.6464129644811623 0.5066951223386589
- link Link3: geometry collision box size=0.9868199680814971 0.8191642077690843 1.3248074473085074; visual box size=0.9868199680814971 0.8191642077690843 1.3248074473085074
- link Link3MinXLink0: geometry collision box size=0.868453233485821 0.8191642077690843 0.9930939669662389; visual box size=0.868453233485821 0.8191642077690843 0.9930939669662389
- link Link3MinXLink1: geometry collision box size=0.5435732949819613 0.7261430293893296 0.5721992542783162; visual box size=0.5435732949819613 0.7261430293893296 0.5721992542783162
- link Link3XLink0: geometry collision box size=0.6948650077809441 0.8191642077690843 0.9134016023189478; visual box size=0.6948650077809441 0.8191642077690843 0.9134016023189478
- link Link3XLink1: geometry collision box size=0.8629667706982338 0.5458716264817558 0.8272876092753887; visual box size=0.8629667706982338 0.5458716264817558 0.8272876092753887
- link Link3ZLink0: geometry collision box size=0.9674333958315764 0.8191642077690843 0.8211407625890506; visual box size=0.9674333958315764 0.8191642077690843 0.8211407625890506
Joints:
- removed joint Link1XLink0_Link1XLink1
- removed joint Link2_Link2ZLink0
- added joint Link1_Link1ZLink0: type revolute, parent Link1, child Link1ZLink0, origin xyz=0 -0.26586621310981307 [0.56988056 0.68133767 0.40105773 0.66240372 0.51845138 0.36966321  0.50366993] rpy=0 0 0, axis 0 0 1, limit lower=-3.14159 upper=3.14159 effort=0.0 velocity=0.0
- added joint Link3XLink1_Link3XLink2: type revolute, parent Link3XLink1, child Link3XLink2, origin xyz=0.8629667706982338 0 0 rpy=0 0 0, axis 1 0 0, limit lower=-3.14159 upper=3.14159 effort=0.0 velocity=0.0
- added joint Link3ZLink0_Link3ZLink1: type revolute, parent Link3ZLink0, child Link3ZLink1, origin xyz=0 0 0.8211407625890506 rpy=0 0 0, axis 0 0 1, limit lower=-3.14159 upper=3.14159 effort=0.0 velocity=0.0
- added joint Link3_Link4: type revolute, parent Link3, child Link4, origin xyz=0 0.8191642077690843 0 rpy=0 0 0, axis 1 0 0, limit lower=-3.14159 upper=3.14159 effort=0.0 velocity=0.0
- added joint Link4MinXLink0_Link4MinXLink1: type revolute, parent Link4MinXLink0, child Link4MinXLink1, origin xyz=-0.5702196198438354 0 0 rpy=0 0 0, axis 1 0 0, limit lower=-3.14159 upper=3.14159 effort=0.0 velocity=0.0
- added joint Link4_Link4MinXLink0: type revolute, parent Link4, child Link4MinXLink0, origin xyz=-0.4022103529998486 0.28622504278677896 0 rpy=0 0 0, axis 1 0 0, limit lower=-3.14159 upper=3.14159 effort=0.0 velocity=0.0
- added joint Link4_Link4XLink0: type revolute, parent Link4, child Link4XLink0, origin xyz=0.4022103529998486 0.28622504278677896 0 rpy=0 0 0, axis 1 0 0, limit lower=-3.14159 upper=3.14159 effort=0.0 velocity=0.0
- added joint Link4_Link4ZLink0: type revolute, parent Link4, child Link4ZLink0, origin xyz=0 -0.28622504278677896 [0.56988056 0.68133767 0.40105773 0.66240372 0.51845138 0.36966321  0.50366993] rpy=0 0 0, axis 0 0 1, limit lower=-3.14159 upper=3.14159 effort=0.0 velocity=0.0
- added joint Link4_Link5: type revolute, parent Link4, child Link5, origin xyz=0 0.5724500855735579 0 rpy=0 0 0, axis 1 0 0, limit lower=-3.14159 upper=3.14159 effort=0.0 velocity=0.0
- added joint Link5_Link5MinXLink0: type revolute, parent Link5, child Link5MinXLink0, origin xyz=-0.6101612854097704 0.4862397246458446 0 rpy=0 0 0, axis 1 0 0, limit lower=-3.14159 upper=3.14159 effort=0.0 velocity=0.0
- added joint Link5_Link5XLink0: type revolute, parent Link5, child Link5XLink0, origin xyz=0.6101612854097704 0.4862397246458446 0 rpy=0 0 0, axis 1 0 0, limit lower=-3.14159 upper=3.14159 effort=0.0 velocity=0.0
- added joint Link5_Link5ZLink0: type revolute, parent Link5, child Link5ZLink0, origin xyz=0 -0.4862397246458446 [0.56988056 0.68133767 0.40105773 0.66240372 0.51845138 0.36966321  0.50366993] rpy=0 0 0, axis 0 0 1, limit lower=-3.14159 upper=3.14159 effort=0.0 velocity=0.0
- joint Link0_Link1: origin xyz=0 0.3079176394835968 0.5602787808363481 rpy=0 0 0 -> xyz=0 0.30668025078934236 0.6813376675078882 rpy=0 0 0
- joint Link1_Link1XLink0: origin xyz=0.435454262077878 0.6741124300356112 0 rpy=0 0 0 -> xyz=0.4123884021814356 0.26586621310981307 0 rpy=0 0 0
- joint Link1_Link2: origin xyz=0 1.3482248600712223 0 rpy=0 0 0 -> xyz=0 0.5317324262196261 0 rpy=0 0 0
- joint Link2_Link2MinXLink0: origin xyz=-0.2932179632766003 0.583778768489682 0 rpy=0 0 0 -> xyz=-0.41428182721214485 0.3232064822405811 0 rpy=0 0 0
- joint Link2_Link2XLink0: origin xyz=0.2932179632766003 0.583778768489682 0 rpy=0 0 0 -> xyz=0.41428182721214485 0.3232064822405811 0 rpy=0 0 0
- joint Link2_Link3: origin xyz=0 1.167557536979364 0 rpy=0 0 0 -> xyz=0 0.6464129644811623 0 rpy=0 0 0
- joint Link3MinXLink0_Link3MinXLink1: origin xyz=-0.9637145854184892 0 0 rpy=0 0 0 -> xyz=-0.868453233485821 0 0 rpy=0 0 0
- joint Link3XLink0_Link3XLink1: origin xyz=0.8896386929508217 0 0 rpy=0 0 0 -> xyz=0.6948650077809441 0 0 rpy=0 0 0
- joint Link3_Link3MinXLink0: origin xyz=-0.5232189047216246 0.6578733749532096 0 rpy=0 0 0 -> xyz=-0.49340998404074854 0.40958210388454214 0 rpy=0 0 0
- joint Link3_Link3XLink0: origin xyz=0.5232189047216246 0.6578733749532096 0 rpy=0 0 0 -> xyz=0.49340998404074854 0.40958210388454214 0 rpy=0 0 0
- joint Link3_Link3ZLink0: origin xyz=0 -0.6578733749532096 [0.3749626  0.38560029 0.56027878 0.50548193 0.35031212] rpy=0 0 0 -> xyz=0 -0.40958210388454214 [0.56988056 0.68133767 0.40105773 0.66240372 0.51845138 0.36966321  0.50366993] rpy=0 0 0

Commit message: color update

File: body.urdf (robot description, URDF)
Before this commit: robot robot, 24 links, 23 joints
Links:
- removed link Link1XLink0
- removed link Link3XLink1
- removed link Link3XLink2
- removed link Link3ZLink1
- removed link Link4MinXLink0
- removed link Link4MinXLink1
- removed link Link5
- removed link Link5MinXLink0
- removed link Link5XLink0
- removed link Link5ZLink0
- added link Link1MinXLink0, mass 1; collision box size=0.7536632007257815 0.5413774461961766 0.7748155204281229; visual box size=0.7536632007257815 0.5413774461961766 0.7748155204281229
- added link Link1MinXLink1, mass 1; collision box size=0.5873819321400094 0.5325917387618954 0.6842928725512087; visual box size=0.5873819321400094 0.5325917387618954 0.6842928725512087
- added link Link1MinXLink2, mass 1; collision box size=0.7194101359958152 0.5325917387618954 0.7639094555910934; visual box size=0.7194101359958152 0.5325917387618954 0.7639094555910934
- added link Link2MinXLink1, mass 1; collision box size=0.9206559773310612 0.6581107295048638 0.8445421404320187; visual box size=0.9206559773310612 0.6581107295048638 0.8445421404320187
- added link Link2MinXLink2, mass 1; collision box size=0.8412494701173248 0.6301648549027135 0.9541664525101754; visual box size=0.8412494701173248 0.6301648549027135 0.9541664525101754
- added link Link2XLink1, mass 1; collision box size=0.8777203760184953 0.6091995047670646 0.8307875095867039; visual box size=0.8777203760184953 0.6091995047670646 0.8307875095867039
- added link Link2ZLink0, mass 1; collision box size=0.6804244855318314 0.8520329897765102 0.8980269994118832; visual box size=0.6804244855318314 0.8520329897765102 0.8980269994118832
- added link Link2ZLink1, mass 1; collision box size=0.6096824261472599 0.5084767837340542 0.6304672467258479; visual box size=0.6096824261472599 0.5084767837340542 0.6304672467258479
- added link Link4XLink1, mass 1; collision box size=0.6665324453701043 0.9097874279213486 0.7127797956152925; visual box size=0.6665324453701043 0.9097874279213486 0.7127797956152925
- link Link0: geometry collision box size=0.7796431096718008 1.4803908126289602 0.5520719426380121; visual box size=0.7796431096718008 1.4803908126289602 0.5520719426380121
- link Link1: geometry collision box size=1.4894160362620865 0.5413774461961766 0.9444937295232064; visual box size=1.4894160362620865 0.5413774461961766 0.9444937295232064
- link Link1ZLink0: geometry collision box size=0.923755826071919 0.5413774461961766 0.7907017902055721; visual box size=0.923755826071919 0.5413774461961766 0.7907017902055721
- link Link2: geometry collision box size=0.8785990718813663 1.2175727448342757 0.7567577937150071; visual box size=0.8785990718813663 1.2175727448342757 0.7567577937150071
- link Link2MinXLink0: geometry collision box size=0.8636615585700008 0.825315725227153 0.874614777712055; visual box size=0.8636615585700008 0.825315725227153 0.874614777712055
- link Link2XLink0: geometry collision box size=0.8228888354232168 0.6091995047670646 0.9997704947729834; visual box size=0.8228888354232168 0.6091995047670646 0.9997704947729834
- link Link3: geometry collision box size=1.1525140958521127 0.5365821129798494 1.054226861736745; visual box size=1.1525140958521127 0.5365821129798494 1.054226861736745
- link Link3MinXLink0: geometry collision box size=0.892939603573799 0.5365821129798494 0.9223403508263248; visual box size=0.892939603573799 0.5365821129798494 0.9223403508263248
- link Link3MinXLink1: geometry collision box size=0.9951637360254411 0.8087834373313934 0.9772073156673399; visual box size=0.9951637360254411 0.8087834373313934 0.9772073156673399
- link Link3XLink0: geometry collision box size=0.965804161349258 0.5365821129798494 0.6743335315432899; visual box size=0.965804161349258 0.5365821129798494 0.6743335315432899
- link Link3ZLink0: geometry collision box size=0.8795200957266596 0.5365821129798494 0.7058796946832526; visual box size=0.8795200957266596 0.5365821129798494 0.7058796946832526
- link Link4: geometry collision box size=1.1294764530085155 1.401526130343834 1.1727887419261445; visual box size=1.1294764530085155 1.401526130343834 1.1727887419261445
- link Link4XLink0: geometry collision box size=0.5641070541188704 0.9288299207725321 0.9440664678801988; visual box size=0.5641070541188704 0.9288299207725321 0.9440664678801988
- link Link4ZLink0: geometry collision box size=0.6957491593937231 0.937617277215913 0.6271564442737183; visual box size=0.6957491593937231 0.937617277215913 0.6271564442737183
Joints:
- removed joint Link1_Link1XLink0
- removed joint Link3XLink0_Link3XLink1
- removed joint Link3XLink1_Link3XLink2
- removed joint Link3ZLink0_Link3ZLink1
- removed joint Link4MinXLink0_Link4MinXLink1
- removed joint Link4_Link4MinXLink0
- removed joint Link4_Link5
- removed joint Link5_Link5MinXLink0
- removed joint Link5_Link5XLink0
- removed joint Link5_Link5ZLink0
- added joint Link1MinXLink0_Link1MinXLink1: type revolute, parent Link1MinXLink0, child Link1MinXLink1, origin xyz=-0.7536632007257815 0 0 rpy=0 0 0, axis 1 0 0, limit lower=-3.14159 upper=3.14159 effort=0.0 velocity=0.0
- added joint Link1MinXLink1_Link1MinXLink2: type revolute, parent Link1MinXLink1, child Link1MinXLink2, origin xyz=-0.5873819321400094 0 0 rpy=0 0 0, axis 1 0 0, limit lower=-3.14159 upper=3.14159 effort=0.0 velocity=0.0
- added joint Link1_Link1MinXLink0: type revolute, parent Link1, child Link1MinXLink0, origin xyz=-0.7447080181310433 0.2706887230980883 0 rpy=0 0 0, axis 1 0 0, limit lower=-3.14159 upper=3.14159 effort=0.0 velocity=0.0
- added joint Link2MinXLink0_Link2MinXLink1: type revolute, parent Link2MinXLink0, child Link2MinXLink1, origin xyz=-0.8636615585700008 0 0 rpy=0 0 0, axis 1 0 0, limit lower=-3.14159 upper=3.14159 effort=0.0 velocity=0.0
- added joint Link2MinXLink1_Link2MinXLink2: type revolute, parent Link2MinXLink1, child Link2MinXLink2, origin xyz=-0.9206559773310612 0 0 rpy=0 0 0, axis 1 0 0, limit lower=-3.14159 upper=3.14159 effort=0.0 velocity=0.0
- added joint Link2XLink0_Link2XLink1: type revolute, parent Link2XLink0, child Link2XLink1, origin xyz=0.8228888354232168 0 0 rpy=0 0 0, axis 1 0 0, limit lower=-3.14159 upper=3.14159 effort=0.0 velocity=0.0
- added joint Link2ZLink0_Link2ZLink1: type revolute, parent Link2ZLink0, child Link2ZLink1, origin xyz=0 0 0.8980269994118832 rpy=0 0 0, axis 0 0 1, limit lower=-3.14159 upper=3.14159 effort=0.0 velocity=0.0
- added joint Link2_Link2ZLink0: type revolute, parent Link2, child Link2ZLink0, origin xyz=0 -0.6087863724171378 [0.27603597 0.47224686 0.3783789  0.52711343 0.58639437 0.52728975] rpy=0 0 0, axis 0 0 1, limit lower=-3.14159 upper=3.14159 effort=0.0 velocity=0.0
- added joint Link4XLink0_Link4XLink1: type revolute, parent Link4XLink0, child Link4XLink1, origin xyz=0.5641070541188704 0 0 rpy=0 0 0, axis 1 0 0, limit lower=-3.14159 upper=3.14159 effort=0.0 velocity=0.0
- joint Link0_Link1: origin xyz=0 0.30668025078934236 0.6813376675078882 rpy=0 0 0 -> xyz=0 0.7401954063144801 0.5863943709630722 rpy=0 0 0
- joint Link1_Link1ZLink0: origin xyz=0 -0.26586621310981307 [0.56988056 0.68133767 0.40105773 0.66240372 0.51845138 0.36966321  0.50366993] rpy=0 0 0 -> xyz=0 -0.2706887230980883 [0.27603597 0.47224686 0.3783789  0.52711343 0.58639437 0.52728975] rpy=0 0 0
- joint Link1_Link2: origin xyz=0 0.5317324262196261 0 rpy=0 0 0 -> xyz=0 0.5413774461961766 0 rpy=0 0 0
- joint Link2_Link2MinXLink0: origin xyz=-0.41428182721214485 0.3232064822405811 0 rpy=0 0 0 -> xyz=-0.43929953594068316 0.6087863724171378 0 rpy=0 0 0
- joint Link2_Link2XLink0: origin xyz=0.41428182721214485 0.3232064822405811 0 rpy=0 0 0 -> xyz=0.43929953594068316 0.6087863724171378 0 rpy=0 0 0
- joint Link2_Link3: origin xyz=0 0.6464129644811623 0 rpy=0 0 0 -> xyz=0 1.2175727448342757 0 rpy=0 0 0
- joint Link3MinXLink0_Link3MinXLink1: origin xyz=-0.868453233485821 0 0 rpy=0 0 0 -> xyz=-0.892939603573799 0 0 rpy=0 0 0
- joint Link3_Link3MinXLink0: origin xyz=-0.49340998404074854 0.40958210388454214 0 rpy=0 0 0 -> xyz=-0.5762570479260564 0.2682910564899247 0 rpy=0 0 0
- joint Link3_Link3XLink0: origin xyz=0.49340998404074854 0.40958210388454214 0 rpy=0 0 0 -> xyz=0.5762570479260564 0.2682910564899247 0 rpy=0 0 0
- joint Link3_Link3ZLink0: origin xyz=0 -0.40958210388454214 [0.56988056 0.68133767 0.40105773 0.66240372 0.51845138 0.36966321  0.50366993] rpy=0 0 0 -> xyz=0 -0.2682910564899247 [0.27603597 0.47224686 0.3783789  0.52711343 0.58639437 0.52728975] rpy=0 0 0
- joint Link3_Link4: origin xyz=0 0.8191642077690843 0 rpy=0 0 0 -> xyz=0 0.5365821129798494 0 rpy=0 0 0
- joint Link4_Link4XLink0: origin xyz=0.4022103529998486 0.28622504278677896 0 rpy=0 0 0 -> xyz=0.5647382265042578 0.700763065171917 0 rpy=0 0 0
- joint Link4_Link4ZLink0: origin xyz=0 -0.28622504278677896 [0.56988056 0.68133767 0.40105773 0.66240372 0.51845138 0.36966321  0.50366993] rpy=0 0 0 -> xyz=0 -0.700763065171917 [0.27603597 0.47224686 0.3783789  0.52711343 0.58639437 0.52728975] rpy=0 0 0
