Commit message: update z joints

File: body.urdf (robot description, URDF)
Before this commit: robot robot, 23 links, 22 joints
Links:
- removed link Link1MinXLink1
- removed link Link1MinXLink2
- removed link Link1ZLink0
- removed link Link2ZLink0
- removed link Link2ZLink1
- removed link Link4XLink0
- removed link Link4XLink1
- removed link Link4ZLink0
- added link Link1XLink0, mass 1; collision box size=0.7343097360622441 0.7895769576654093 0.8441214191816651; visual box size=0.7343097360622441 0.7895769576654093 0.8441214191816651
- added link Link3MinXLink2, mass 1; collision box size=0.9032974547407937 0.8178514260974935 0.793559982470319; visual box size=0.9032974547407937 0.8178514260974935 0.793559982470319
- added link Link3XLink1, mass 1; collision box size=0.9935212630828492 0.64017390791797 0.8317572522993979; visual box size=0.9935212630828492 0.64017390791797 0.8317572522993979
- added link Link5, mass 1; collision box size=0.7737275817612951 1.4865253365598898 1.242145228318634; visual box size=0.7737275817612951 1.4865253365598898 1.242145228318634
- added link Link5ZLink0, mass 1; collision box size=0.7737275817612951 0.9551286093340141 0.8163085174509247; visual box size=0.7737275817612951 0.9551286093340141 0.8163085174509247
- link Link0: geometry collision box size=1.3738284973141908 0.6555284085930438 1.2533950571735744; visual box size=1.3738284973141908 0.6555284085930438 1.2533950571735744
- link Link1: geometry collision box size=1.3818194746754153 1.2992918815233505 0.6786436865100399; visual box size=1.3818194746754153 1.2992918815233505 0.6786436865100399
- link Link1MinXLink0: geometry collision box size=0.6151451919071614 0.5929110414452032 0.8621082960935451; visual box size=0.6151451919071614 0.5929110414452032 0.8621082960935451
- link Link2: geometry collision box size=0.5873608025587613 1.0613148698731907 1.280944175066678; visual box size=0.5873608025587613 1.0613148698731907 1.280944175066678
- link Link2MinXLink0: geometry collision box size=0.7318136385303389 0.81780696782711 0.5349129818706551; visual box size=0.7318136385303389 0.81780696782711 0.5349129818706551
- link Link2MinXLink1: geometry collision box size=0.6016279074872914 0.81780696782711 0.8094584648628036; visual box size=0.6016279074872914 0.81780696782711 0.8094584648628036
- link Link2MinXLink2: geometry collision box size=0.9926614129835312 0.9413576620137811 0.529660517695571; visual box size=0.9926614129835312 0.9413576620137811 0.529660517695571
- link Link2XLink0: geometry collision box size=0.7036736256937897 0.5467602146822516 0.8193781110103167; visual box size=0.7036736256937897 0.5467602146822516 0.8193781110103167
- link Link2XLink1: geometry collision box size=0.8076247123835192 0.5467602146822516 0.8414725395088738; visual box size=0.8076247123835192 0.5467602146822516 0.8414725395088738
- link Link3: geometry collision box size=0.8816958192693513 1.455557378856081 0.8985667136999128; visual box size=0.8816958192693513 1.455557378856081 0.8985667136999128
- link Link3MinXLink0: geometry collision box size=0.9863980455454617 0.8672633685047536 0.6524408822311505; visual box size=0.9863980455454617 0.8672633685047536 0.6524408822311505
- link Link3MinXLink1: geometry collision box size=0.9738694952541364 0.8178514260974935 0.6319377898391219; visual box size=0.9738694952541364 0.8178514260974935 0.6319377898391219
- link Link3XLink0: geometry collision box size=0.8167854068151932 0.8692372375101611 0.5020576495747486; visual box size=0.8167854068151932 0.8692372375101611 0.5020576495747486
- link Link3ZLink0: geometry collision box size=0.8816958192693513 0.9850558203672419 0.6250332174486661; visual box size=0.8816958192693513 0.9850558203672419 0.6250332174486661
- link Link4: geometry collision box size=0.8966778633396246 1.2614779982101536 0.820477330249176; visual box size=0.8966778633396246 1.2614779982101536 0.820477330249176
Joints:
- removed joint Link1MinXLink0_Link1MinXLink1
- removed joint Link1MinXLink1_Link1MinXLink2
- removed joint Link1_Link1ZLink0
- removed joint Link2ZLink0_Link2ZLink1
- removed joint Link2_Link2ZLink0
- removed joint Link4XLink0_Link4XLink1
- removed joint Link4_Link4XLink0
- removed joint Link4_Link4ZLink0
- added joint Link1_Link1XLink0: type revolute, parent Link1, child Link1XLink0, origin xyz=0.6909097373377077 0.6496459407616753 0 rpy=0 0 0, axis 1 0 0, limit lower=-3.14159 upper=3.14159 effort=0.0 velocity=0.0
- added joint Link3MinXLink1_Link3MinXLink2: type revolute, parent Link3MinXLink1, child Link3MinXLink2, origin xyz=-0.9738694952541364 0 0 rpy=0 0 0, axis 1 0 0, limit lower=-3.14159 upper=3.14159 effort=0.0 velocity=0.0
- added joint Link3XLink0_Link3XLink1: type revolute, parent Link3XLink0, child Link3XLink1, origin xyz=0.8167854068151932 0 0 rpy=0 0 0, axis 1 0 0, limit lower=-3.14159 upper=3.14159 effort=0.0 velocity=0.0
- added joint Link4_Link5: type revolute, parent Link4, child Link5, origin xyz=0 1.2614779982101536 0 rpy=0 0 0, axis 1 0 0, limit lower=-3.14159 upper=3.14159 effort=0.0 velocity=0.0
- added joint Link5_Link5ZLink0: type revolute, parent Link5, child Link5ZLink0, origin xyz=0 0.7432626682799449 0.621072614159317 rpy=0 0 0, axis 0 0 1, limit lower=-3.14159 upper=3.14159 effort=0.0 velocity=0.0
- joint Link0_Link1: origin xyz=0 0.7401954063144801 0.5863943709630722 rpy=0 0 0 -> xyz=0 0.3277642042965219 0.640472087533339 rpy=0 0 0
- joint Link1_Link1MinXLink0: origin xyz=-0.7447080181310433 0.2706887230980883 0 rpy=0 0 0 -> xyz=-0.6909097373377077 0.6496459407616753 0 rpy=0 0 0
- joint Link1_Link2: origin xyz=0 0.5413774461961766 0 rpy=0 0 0 -> xyz=0 1.2992918815233505 0 rpy=0 0 0
- joint Link2MinXLink0_Link2MinXLink1: origin xyz=-0.8636615585700008 0 0 rpy=0 0 0 -> xyz=-0.7318136385303389 0 0 rpy=0 0 0
- joint Link2MinXLink1_Link2MinXLink2: origin xyz=-0.9206559773310612 0 0 rpy=0 0 0 -> xyz=-0.6016279074872914 0 0 rpy=0 0 0
- joint Link2XLink0_Link2XLink1: origin xyz=0.8228888354232168 0 0 rpy=0 0 0 -> xyz=0.7036736256937897 0 0 rpy=0 0 0
- joint Link2_Link2MinXLink0: origin xyz=-0.43929953594068316 0.6087863724171378 0 rpy=0 0 0 -> xyz=-0.29368040127938067 0.5306574349365953 0 rpy=0 0 0
- joint Link2_Link2XLink0: origin xyz=0.43929953594068316 0.6087863724171378 0 rpy=0 0 0 -> xyz=0.29368040127938067 0.5306574349365953 0 rpy=0 0 0
- joint Link2_Link3: origin xyz=0 1.2175727448342757 0 rpy=0 0 0 -> xyz=0 1.0613148698731907 0 rpy=0 0 0
- joint Link3MinXLink0_Link3MinXLink1: origin xyz=-0.892939603573799 0 0 rpy=0 0 0 -> xyz=-0.9863980455454617 0 0 rpy=0 0 0
- joint Link3_Link3MinXLink0: origin xyz=-0.5762570479260564 0.2682910564899247 0 rpy=0 0 0 -> xyz=-0.4408479096346756 0.7277786894280405 0 rpy=0 0 0
- joint Link3_Link3XLink0: origin xyz=0.5762570479260564 0.2682910564899247 0 rpy=0 0 0 -> xyz=0.4408479096346756 0.7277786894280405 0 rpy=0 0 0
- joint Link3_Link3ZLink0: origin xyz=0 -0.2682910564899247 [0.27603597 0.47224686 0.3783789  0.52711343 0.58639437 0.52728975] rpy=0 0 0 -> xyz=0 0.7277786894280405 0.4492833568499564 rpy=0 0 0
- joint Link3_Link4: origin xyz=0 0.5365821129798494 0 rpy=0 0 0 -> xyz=0 1.455557378856081 0 rpy=0 0 0

Commit message: refactoring

File: body.urdf (robot description, URDF)
Before this commit: robot robot, 20 links, 19 joints
Links:
- removed link Link1XLink0
- removed link Link2MinXLink0
- removed link Link2MinXLink1
- removed link Link2MinXLink2
- removed link Link3
- removed link Link3MinXLink0
- removed link Link3MinXLink1
- removed link Link3MinXLink2
- removed link Link3XLink0
- removed link Link3XLink1
- removed link Link3ZLink0
- removed link Link4
- removed link Link5
- removed link Link5ZLink0
- added link Link1MinXLink1, mass 1; collision box size=0.5229804737996324 0.8384767929953454 0.875556463449984; visual box size=0.5229804737996324 0.8384767929953454 0.875556463449984
- added link Link1ZLink0, mass 1; collision box size=0.8598286407542761 0.52268695217379 0.8539409923405592; visual box size=0.8598286407542761 0.52268695217379 0.8539409923405592
- added link Link1ZLink1, mass 1; collision box size=0.7243664259859752 0.52268695217379 0.8220106956711238; visual box size=0.7243664259859752 0.52268695217379 0.8220106956711238
- link Link0: geometry collision box size=0.9511106651797404 0.6493523724012363 1.3370444374668118; visual box size=0.9511106651797404 0.6493523724012363 1.3370444374668118
- link Link1: geometry collision box size=1.1201742907588086 0.8127133059338928 0.9044584576413319; visual box size=1.1201742907588086 0.8127133059338928 0.9044584576413319
- link Link1MinXLink0: geometry collision box size=0.8730056316504758 0.8127133059338928 0.9924966515813225; visual box size=0.8730056316504758 0.8127133059338928 0.9924966515813225
- link Link2: geometry collision box size=1.3178582897358964 0.5497047138812728 0.5314710982427203; visual box size=1.3178582897358964 0.5497047138812728 0.5314710982427203
- link Link2XLink0: geometry collision box size=0.9321001058015786 0.5497047138812728 0.9819936177516299; visual box size=0.9321001058015786 0.5497047138812728 0.9819936177516299
- link Link2XLink1: geometry collision box size=0.7823182213003526 0.9156659023098404 0.861017076888723; visual box size=0.7823182213003526 0.9156659023098404 0.861017076888723
Joints:
- removed joint Link1_Link1XLink0
- removed joint Link2MinXLink0_Link2MinXLink1
- removed joint Link2MinXLink1_Link2MinXLink2
- removed joint Link2_Link2MinXLink0
- removed joint Link2_Link3
- removed joint Link3MinXLink0_Link3MinXLink1
- removed joint Link3MinXLink1_Link3MinXLink2
- removed joint Link3XLink0_Link3XLink1
- removed joint Link3_Link3MinXLink0
- removed joint Link3_Link3XLink0
- removed joint Link3_Link3ZLink0
- removed joint Link3_Link4
- removed joint Link4_Link5
- removed joint Link5_Link5ZLink0
- added joint Link1MinXLink0_Link1MinXLink1: type revolute, parent Link1MinXLink0, child Link1MinXLink1, origin xyz=-0.8730056316504758 0 0 rpy=0 0 0, axis 1 0 0, limit lower=-3.14159 upper=3.14159 effort=0.0 velocity=0.0
- added joint Link1ZLink0_Link1ZLink1: type revolute, parent Link1ZLink0, child Link1ZLink1, origin xyz=0 0 0.8539409923405592 rpy=0 0 0, axis 0 0 1, limit lower=-3.14159 upper=3.14159 effort=0.0 velocity=0.0
- added joint Link1_Link1ZLink0: type revolute, parent Link1, child Link1ZLink0, origin xyz=0 0.4063566529669464 0.45222922882066596 rpy=0 0 0, axis 0 0 1, limit lower=-3.14159 upper=3.14159 effort=0.0 velocity=0.0
- joint Link0_Link1: origin xyz=0 0.3277642042965219 0.640472087533339 rpy=0 0 0 -> xyz=0 0.32467618620061817 0.6991342758684187 rpy=0 0 0
- joint Link1_Link1MinXLink0: origin xyz=-0.6909097373377077 0.6496459407616753 0 rpy=0 0 0 -> xyz=-0.5600871453794043 0.4063566529669464 0 rpy=0 0 0
- joint Link1_Link2: origin xyz=0 1.2992918815233505 0 rpy=0 0 0 -> xyz=0 0.8127133059338928 0 rpy=0 0 0
- joint Link2XLink0_Link2XLink1: origin xyz=0.7036736256937897 0 0 rpy=0 0 0 -> xyz=0.9321001058015786 0 0 rpy=0 0 0
- joint Link2_Link2XLink0: origin xyz=0.29368040127938067 0.5306574349365953 0 rpy=0 0 0 -> xyz=0.6589291448679482 0.2748523569406364 0 rpy=0 0 0

Commit message: refactoring

File: body.urdf (robot description, URDF)
Before this commit: robot robot, 9 links, 8 joints
Links:
- added link Link1MinXLink2, mass 1; collision box size=0.7519271100136891 0.6328787402042939 0.906606198083527; visual box size=0.7519271100136891 0.6328787402042939 0.906606198083527
- added link Link1XLink0, mass 1; collision box size=0.79059714119881 0.7926847716472583 0.7220776960386861; visual box size=0.79059714119881 0.7926847716472583 0.7220776960386861
- added link Link1XLink1, mass 1; collision box size=0.5331398404602268 0.7926847716472583 0.5374202058426159; visual box size=0.5331398404602268 0.7926847716472583 0.5374202058426159
- added link Link2MinXLink0, mass 1; collision box size=0.5258509544115282 0.8736150137389163 0.8223963184742477; visual box size=0.5258509544115282 0.8736150137389163 0.8223963184742477
- added link Link2MinXLink1, mass 1; collision box size=0.9044787534565693 0.700871894254916 0.8246712576575725; visual box size=0.9044787534565693 0.700871894254916 0.8246712576575725
- added link Link2ZLink0, mass 1; collision box size=0.7757844850169042 0.9297488359156825 0.992602116219882; visual box size=0.7757844850169042 0.9297488359156825 0.992602116219882
- added link Link3, mass 1; collision box size=0.8654096662132406 0.8613816842851366 1.4148571338104872; visual box size=0.8654096662132406 0.8613816842851366 1.4148571338104872
- added link Link3MinXLink0, mass 1; collision box size=0.597267374488458 0.842613979288303 0.9405303662346394; visual box size=0.597267374488458 0.842613979288303 0.9405303662346394
- added link Link3XLink0, mass 1; collision box size=0.7766249005600732 0.8613816842851366 0.8769460912645786; visual box size=0.7766249005600732 0.8613816842851366 0.8769460912645786
- added link Link3XLink1, mass 1; collision box size=0.5422980061564838 0.7865808799889833 0.7706102855915178; visual box size=0.5422980061564838 0.7865808799889833 0.7706102855915178
- added link Link3XLink2, mass 1; collision box size=0.618521231873784 0.7865808799889833 0.7343863157262899; visual box size=0.618521231873784 0.7865808799889833 0.7343863157262899
- added link Link3ZLink0, mass 1; collision box size=0.6389131337976612 0.7793205562369538 0.5340105640171879; visual box size=0.6389131337976612 0.7793205562369538 0.5340105640171879
- added link Link4, mass 1; collision box size=1.4802012976705194 0.7452844430038866 1.3871066845375788; visual box size=1.4802012976705194 0.7452844430038866 1.3871066845375788
- added link Link4XLink0, mass 1; collision box size=0.6801385390015214 0.7452844430038866 0.665897399833113; visual box size=0.6801385390015214 0.7452844430038866 0.665897399833113
- added link Link4XLink1, mass 1; collision box size=0.6019341132028897 0.7800749496453965 0.7375422685076158; visual box size=0.6019341132028897 0.7800749496453965 0.7375422685076158
- added link Link4XLink2, mass 1; collision box size=0.6873595942917341 0.6162483919556425 0.7084080738584637; visual box size=0.6873595942917341 0.6162483919556425 0.7084080738584637
- added link Link4ZLink0, mass 1; collision box size=0.8143161575201224 0.5531045013702438 0.9599363740976146; visual box size=0.8143161575201224 0.5531045013702438 0.9599363740976146
- added link Link4ZLink1, mass 1; collision box size=0.7329546028998921 0.5531045013702438 0.7779301419533065; visual box size=0.7329546028998921 0.5531045013702438 0.7779301419533065
- link Link0: geometry collision box size=0.536243132567079 1.4177334892630449 1.2748863051889014; visual box size=0.536243132567079 1.4177334892630449 1.2748863051889014
- link Link1: geometry collision box size=0.7529151162627209 1.3784397229640537 1.479013873595349; visual box size=0.7529151162627209 1.3784397229640537 1.479013873595349
- link Link1MinXLink0: geometry collision box size=0.7050834046224055 0.8936639809611566 0.6575066030459008; visual box size=0.7050834046224055 0.8936639809611566 0.6575066030459008
- link Link1MinXLink1: geometry collision box size=0.7751192717473616 0.6328787402042939 0.9235017504877954; visual box size=0.7751192717473616 0.6328787402042939 0.9235017504877954
- link Link1ZLink0: geometry collision box size=0.6264801929530979 0.770625433158777 0.7823140756981668; visual box size=0.6264801929530979 0.770625433158777 0.7823140756981668
- link Link1ZLink1: geometry collision box size=0.6078824720040921 0.58040488633511 0.5536710051814991; visual box size=0.6078824720040921 0.58040488633511 0.5536710051814991
- link Link2: geometry collision box size=1.0824255721267064 1.3079998499888732 0.6681351668687164; visual box size=1.0824255721267064 1.3079998499888732 0.6681351668687164
- link Link2XLink0: geometry collision box size=0.8419557552268331 0.5389516662694596 0.5770588979453601; visual box size=0.8419557552268331 0.5389516662694596 0.5770588979453601
- link Link2XLink1: geometry collision box size=0.7396609768909403 0.5389516662694596 0.6933914861122759; visual box size=0.7396609768909403 0.5389516662694596 0.6933914861122759
Joints:
- added joint Link1MinXLink1_Link1MinXLink2: type revolute, parent Link1MinXLink1, child Link1MinXLink2, origin xyz=-0.7751192717473616 0 0 rpy=0 0 0, axis 1 0 0, limit lower=-3.14159 upper=3.14159 effort=0.0 velocity=0.0
- added joint Link1XLink0_Link1XLink1: type revolute, parent Link1XLink0, child Link1XLink1, origin xyz=0.79059714119881 0 0 rpy=0 0 0, axis 1 0 0, limit lower=-3.14159 upper=3.14159 effort=0.0 velocity=0.0
- added joint Link1_Link1XLink0: type revolute, parent Link1, child Link1XLink0, origin xyz=0.37645755813136045 0.6892198614820269 0 rpy=0 0 0, axis 1 0 0, limit lower=-3.14159 upper=3.14159 effort=0.0 velocity=0.0
- added joint Link2MinXLink0_Link2MinXLink1: type revolute, parent Link2MinXLink0, child Link2MinXLink1, origin xyz=-0.5258509544115282 0 0 rpy=0 0 0, axis 1 0 0, limit lower=-3.14159 upper=3.14159 effort=0.0 velocity=0.0
- added joint Link2_Link2MinXLink0: type revolute, parent Link2, child Link2MinXLink0, origin xyz=-0.5412127860633532 0.6539999249944366 0 rpy=0 0 0, axis 1 0 0, limit lower=-3.14159 upper=3.14159 effort=0.0 velocity=0.0
- added joint Link2_Link2ZLink0: type revolute, parent Link2, child Link2ZLink0, origin xyz=0 0.6539999249944366 0.3340675834343582 rpy=0 0 0, axis 0 0 1, limit lower=-3.14159 upper=3.14159 effort=0.0 velocity=0.0
- added joint Link2_Link3: type revolute, parent Link2, child Link3, origin xyz=0 1.3079998499888732 0 rpy=0 0 0, axis 1 0 0, limit lower=-3.14159 upper=3.14159 effort=0.0 velocity=0.0
- added joint Link3XLink0_Link3XLink1: type revolute, parent Link3XLink0, child Link3XLink1, origin xyz=0.7766249005600732 0 0 rpy=0 0 0, axis 1 0 0, limit lower=-3.14159 upper=3.14159 effort=0.0 velocity=0.0
- added joint Link3XLink1_Link3XLink2: type revolute, parent Link3XLink1, child Link3XLink2, origin xyz=0.5422980061564838 0 0 rpy=0 0 0, axis 1 0 0, limit lower=-3.14159 upper=3.14159 effort=0.0 velocity=0.0
- added joint Link3_Link3MinXLink0: type revolute, parent Link3, child Link3MinXLink0, origin xyz=-0.4327048331066203 0.4306908421425683 0 rpy=0 0 0, axis 1 0 0, limit lower=-3.14159 upper=3.14159 effort=0.0 velocity=0.0
- added joint Link3_Link3XLink0: type revolute, parent Link3, child Link3XLink0, origin xyz=0.4327048331066203 0.4306908421425683 0 rpy=0 0 0, axis 1 0 0, limit lower=-3.14159 upper=3.14159 effort=0.0 velocity=0.0
- added joint Link3_Link3ZLink0: type revolute, parent Link3, child Link3ZLink0, origin xyz=0 0.4306908421425683 0.7074285669052436 rpy=0 0 0, axis 0 0 1, limit lower=-3.14159 upper=3.14159 effort=0.0 velocity=0.0
- added joint Link3_Link4: type revolute, parent Link3, child Link4, origin xyz=0 0.8613816842851366 0 rpy=0 0 0, axis 1 0 0, limit lower=-3.14159 upper=3.14159 effort=0.0 velocity=0.0
- added joint Link4XLink0_Link4XLink1: type revolute, parent Link4XLink0, child Link4XLink1, origin xyz=0.6801385390015214 0 0 rpy=0 0 0, axis 1 0 0, limit lower=-3.14159 upper=3.14159 effort=0.0 velocity=0.0
- added joint Link4XLink1_Link4XLink2: type revolute, parent Link4XLink1, child Link4XLink2, origin xyz=0.6019341132028897 0 0 rpy=0 0 0, axis 1 0 0, limit lower=-3.14159 upper=3.14159 effort=0.0 velocity=0.0
- added joint Link4ZLink0_Link4ZLink1: type revolute, parent Link4ZLink0, child Link4ZLink1, origin xyz=0 0 0.9599363740976146 rpy=0 0 0, axis 0 0 1, limit lower=-3.14159 upper=3.14159 effort=0.0 velocity=0.0
- added joint Link4_Link4XLink0: type revolute, parent Link4, child Link4XLink0, origin xyz=0.7401006488352597 0.3726422215019433 0 rpy=0 0 0, axis 1 0 0, limit lower=-3.14159 upper=3.14159 effort=0.0 velocity=0.0
- added joint Link4_Link4ZLink0: type revolute, parent Link4, child Link4ZLink0, origin xyz=0 0.3726422215019433 0.6935533422687894 rpy=0 0 0, axis 0 0 1, limit lower=-3.14159 upper=3.14159 effort=0.0 velocity=0.0
- joint Link0_Link1: origin xyz=0 0.32467618620061817 0.6991342758684187 rpy=0 0 0 -> xyz=0 0.7088667446315224 0.7395069367976745 rpy=0 0 0
- joint Link1MinXLink0_Link1MinXLink1: origin xyz=-0.8730056316504758 0 0 rpy=0 0 0 -> xyz=-0.7050834046224055 0 0 rpy=0 0 0
- joint Link1ZLink0_Link1ZLink1: origin xyz=0 0 0.8539409923405592 rpy=0 0 0 -> xyz=0 0 0.7823140756981668 rpy=0 0 0
- joint Link1_Link1MinXLink0: origin xyz=-0.5600871453794043 0.4063566529669464 0 rpy=0 0 0 -> xyz=-0.37645755813136045 0.6892198614820269 0 rpy=0 0 0
- joint Link1_Link1ZLink0: origin xyz=0 0.4063566529669464 0.45222922882066596 rpy=0 0 0 -> xyz=0 0.6892198614820269 0.7395069367976745 rpy=0 0 0
- joint Link1_Link2: origin xyz=0 0.8127133059338928 0 rpy=0 0 0 -> xyz=0 1.3784397229640537 0 rpy=0 0 0
- joint Link2XLink0_Link2XLink1: origin xyz=0.9321001058015786 0 0 rpy=0 0 0 -> xyz=0.8419557552268331 0 0 rpy=0 0 0
- joint Link2_Link2XLink0: origin xyz=0.6589291448679482 0.2748523569406364 0 rpy=0 0 0 -> xyz=0.5412127860633532 0.6539999249944366 0 rpy=0 0 0
