Commit message: big refactor

File: body.urdf (robot description, URDF)
Before this commit: robot robot, 27 links, 26 joints
Links:
- removed link Link1MinXLink0
- removed link Link1MinXLink1
- removed link Link1MinXLink2
- removed link Link1ZLink0
- removed link Link1ZLink1
- removed link Link2MinXLink0
- removed link Link2MinXLink1
- removed link Link2XLink0
- removed link Link2XLink1
- removed link Link4XLink1
- removed link Link4XLink2
- added link Link2ZLink1, mass 1; collision box size=0.665181488470747 0.7865983864026465 0.5434970791927716; visual box size=0.665181488470747 0.7865983864026465 0.5434970791927716
- added link Link3ZLink1, mass 1; collision box size=0.5282374429066727 0.7120527819933724 0.822373924984763; visual box size=0.5282374429066727 0.7120527819933724 0.822373924984763
- added link Link4MinXLink0, mass 1; collision box size=0.5304852067534422 0.6085139608468063 0.6673852596207518; visual box size=0.5304852067534422 0.6085139608468063 0.6673852596207518
- added link Link5, mass 1; collision box size=1.298093002316262 0.9388658141124661 0.9663934357247247; visual box size=1.298093002316262 0.9388658141124661 0.9663934357247247
- added link Link5MinXLink0, mass 1; collision box size=0.8058972244348794 0.624845408685738 0.7345735297027745; visual box size=0.8058972244348794 0.624845408685738 0.7345735297027745
- added link Link5MinXLink1, mass 1; collision box size=0.8058972244348794 0.624845408685738 0.7345735297027745; visual box size=0.8058972244348794 0.624845408685738 0.7345735297027745
- added link Link5MinXLink2, mass 1; collision box size=0.8058972244348794 0.624845408685738 0.7345735297027745; visual box size=0.8058972244348794 0.624845408685738 0.7345735297027745
- added link Link5XLink0, mass 1; collision box size=0.7666356266935199 0.8909402156274544 0.5995804216090428; visual box size=0.7666356266935199 0.8909402156274544 0.5995804216090428
- added link Link5XLink1, mass 1; collision box size=0.7666356266935199 0.8909402156274544 0.5995804216090428; visual box size=0.7666356266935199 0.8909402156274544 0.5995804216090428
- added link Link5XLink2, mass 1; collision box size=0.7666356266935199 0.8909402156274544 0.5995804216090428; visual box size=0.7666356266935199 0.8909402156274544 0.5995804216090428
- added link Link5ZLink0, mass 1; collision box size=0.6789275874989416 0.5085989123918809 0.8706558319717685; visual box size=0.6789275874989416 0.5085989123918809 0.8706558319717685
- link Link0: geometry collision box size=1.4673137424944365 0.6017433728464265 1.4746439739223156; visual box size=1.4673137424944365 0.6017433728464265 1.4746439739223156
- link Link1: geometry collision box size=1.4667591108501912 0.8781129826073822 1.2261635513491613; visual box size=1.4667591108501912 0.8781129826073822 1.2261635513491613
- link Link1XLink0: geometry collision box size=0.5889040860224526 0.8337623649445782 0.5625402022424616; visual box size=0.5889040860224526 0.8337623649445782 0.5625402022424616
- link Link1XLink1: geometry collision box size=0.5889040860224526 0.8337623649445782 0.5625402022424616; visual box size=0.5889040860224526 0.8337623649445782 0.5625402022424616
- link Link2: geometry collision box size=0.8252150030152644 0.5849654264192427 0.9199074025726298; visual box size=0.8252150030152644 0.5849654264192427 0.9199074025726298
- link Link2ZLink0: geometry collision box size=0.665181488470747 0.5849654264192427 0.5434970791927716; visual box size=0.665181488470747 0.5849654264192427 0.5434970791927716
- link Link3: geometry collision box size=0.5646903749954357 0.7474666128173686 0.7086240024657914; visual box size=0.5646903749954357 0.7474666128173686 0.7086240024657914
- link Link3MinXLink0: geometry collision box size=0.9090199822996068 0.6204220288010995 0.8414736955431559; visual box size=0.9090199822996068 0.6204220288010995 0.8414736955431559
- link Link3XLink0: geometry collision box size=0.7618081682573982 0.602096749154368 0.9837510440125012; visual box size=0.7618081682573982 0.602096749154368 0.9837510440125012
- link Link3XLink1: geometry collision box size=0.7618081682573982 0.602096749154368 0.9837510440125012; visual box size=0.7618081682573982 0.602096749154368 0.9837510440125012
- link Link3XLink2: geometry collision box size=0.7618081682573982 0.602096749154368 0.9837510440125012; visual box size=0.7618081682573982 0.602096749154368 0.9837510440125012
- link Link3ZLink0: geometry collision box size=0.5282374429066727 0.7120527819933724 0.822373924984763; visual box size=0.5282374429066727 0.7120527819933724 0.822373924984763
- link Link4: geometry collision box size=1.4005061972957198 0.6085139608468063 1.3753320353360985; visual box size=1.4005061972957198 0.6085139608468063 1.3753320353360985
- link Link4XLink0: geometry collision box size=0.7970239975650404 0.6085139608468063 0.7156851964367557; visual box size=0.7970239975650404 0.6085139608468063 0.7156851964367557
- link Link4ZLink0: geometry collision box size=0.8848177128364187 0.6085139608468063 0.7181397206658644; visual box size=0.8848177128364187 0.6085139608468063 0.7181397206658644
- link Link4ZLink1: geometry collision box size=0.8848177128364187 0.8399421967244383 0.7181397206658644; visual box size=0.8848177128364187 0.8399421967244383 0.7181397206658644
Joints:
- removed joint Link1MinXLink0_Link1MinXLink1
- removed joint Link1MinXLink1_Link1MinXLink2
- removed joint Link1ZLink0_Link1ZLink1
- removed joint Link1_Link1MinXLink0
- removed joint Link1_Link1ZLink0
- removed joint Link2MinXLink0_Link2MinXLink1
- removed joint Link2XLink0_Link2XLink1
- removed joint Link2_Link2MinXLink0
- removed joint Link2_Link2XLink0
- removed joint Link4XLink0_Link4XLink1
- removed joint Link4XLink1_Link4XLink2
- added joint Link2ZLink0_Link2ZLink1: type revolute, parent Link2ZLink0, child Link2ZLink1, origin xyz=0 0 0.5434970791927716 rpy=0 0 0, axis 0 0 1, limit lower=-3.14159 upper=3.14159 effort=0.0 velocity=0.0
- added joint Link3ZLink0_Link3ZLink1: type revolute, parent Link3ZLink0, child Link3ZLink1, origin xyz=0 0 0.822373924984763 rpy=0 0 0, axis 0 0 1, limit lower=-3.14159 upper=3.14159 effort=0.0 velocity=0.0
- added joint Link4_Link4MinXLink0: type revolute, parent Link4, child Link4MinXLink0, origin xyz=-0.7002530986478599 0.30425698042340316 0 rpy=0 0 0, axis 1 0 0, limit lower=-3.14159 upper=3.14159 effort=0.0 velocity=0.0
- added joint Link4_Link5: type revolute, parent Link4, child Link5, origin xyz=0 0.6085139608468063 0 rpy=0 0 0, axis 1 0 0, limit lower=-3.14159 upper=3.14159 effort=0.0 velocity=0.0
- added joint Link5MinXLink0_Link5MinXLink1: type revolute, parent Link5MinXLink0, child Link5MinXLink1, origin xyz=-0.8058972244348794 0 0 rpy=0 0 0, axis 1 0 0, limit lower=-3.14159 upper=3.14159 effort=0.0 velocity=0.0
- added joint Link5MinXLink1_Link5MinXLink2: type revolute, parent Link5MinXLink1, child Link5MinXLink2, origin xyz=-0.8058972244348794 0 0 rpy=0 0 0, axis 1 0 0, limit lower=-3.14159 upper=3.14159 effort=0.0 velocity=0.0
- added joint Link5XLink0_Link5XLink1: type revolute, parent Link5XLink0, child Link5XLink1, origin xyz=0.7666356266935199 0 0 rpy=0 0 0, axis 1 0 0, limit lower=-3.14159 upper=3.14159 effort=0.0 velocity=0.0
- added joint Link5XLink1_Link5XLink2: type revolute, parent Link5XLink1, child Link5XLink2, origin xyz=0.7666356266935199 0 0 rpy=0 0 0, axis 1 0 0, limit lower=-3.14159 upper=3.14159 effort=0.0 velocity=0.0
- added joint Link5_Link5MinXLink0: type revolute, parent Link5, child Link5MinXLink0, origin xyz=-0.649046501158131 0.46943290705623303 0 rpy=0 0 0, axis 1 0 0, limit lower=-3.14159 upper=3.14159 effort=0.0 velocity=0.0
- added joint Link5_Link5XLink0: type revolute, parent Link5, child Link5XLink0, origin xyz=0.649046501158131 0.46943290705623303 0 rpy=0 0 0, axis 1 0 0, limit lower=-3.14159 upper=3.14159 effort=0.0 velocity=0.0
- added joint Link5_Link5ZLink0: type revolute, parent Link5, child Link5ZLink0, origin xyz=0 0.46943290705623303 0.48319671786236235 rpy=0 0 0, axis 0 0 1, limit lower=-3.14159 upper=3.14159 effort=0.0 velocity=0.0
- joint Link0_Link1: origin xyz=0 0.7088667446315224 0.7395069367976745 rpy=0 0 0 -> xyz=0 0.30087168642321327 0.7373219869611578 rpy=0 0 0
- joint Link1XLink0_Link1XLink1: origin xyz=0.79059714119881 0 0 rpy=0 0 0 -> xyz=0.5889040860224526 0 0 rpy=0 0 0
- joint Link1_Link1XLink0: origin xyz=0.37645755813136045 0.6892198614820269 0 rpy=0 0 0 -> xyz=0.7333795554250956 0.4390564913036911 0 rpy=0 0 0
- joint Link1_Link2: origin xyz=0 1.3784397229640537 0 rpy=0 0 0 -> xyz=0 0.8781129826073822 0 rpy=0 0 0
- joint Link2_Link2ZLink0: origin xyz=0 0.6539999249944366 0.3340675834343582 rpy=0 0 0 -> xyz=0 0.2924827132096213 0.4599537012863149 rpy=0 0 0
- joint Link2_Link3: origin xyz=0 1.3079998499888732 0 rpy=0 0 0 -> xyz=0 0.5849654264192427 0 rpy=0 0 0
- joint Link3XLink0_Link3XLink1: origin xyz=0.7766249005600732 0 0 rpy=0 0 0 -> xyz=0.7618081682573982 0 0 rpy=0 0 0
- joint Link3XLink1_Link3XLink2: origin xyz=0.5422980061564838 0 0 rpy=0 0 0 -> xyz=0.7618081682573982 0 0 rpy=0 0 0
- joint Link3_Link3MinXLink0: origin xyz=-0.4327048331066203 0.4306908421425683 0 rpy=0 0 0 -> xyz=-0.28234518749771786 0.3737333064086843 0 rpy=0 0 0
- joint Link3_Link3XLink0: origin xyz=0.4327048331066203 0.4306908421425683 0 rpy=0 0 0 -> xyz=0.28234518749771786 0.3737333064086843 0 rpy=0 0 0
- joint Link3_Link3ZLink0: origin xyz=0 0.4306908421425683 0.7074285669052436 rpy=0 0 0 -> xyz=0 0.3737333064086843 0.3543120012328957 rpy=0 0 0
- joint Link3_Link4: origin xyz=0 0.8613816842851366 0 rpy=0 0 0 -> xyz=0 0.7474666128173686 0 rpy=0 0 0
- joint Link4ZLink0_Link4ZLink1: origin xyz=0 0 0.9599363740976146 rpy=0 0 0 -> xyz=0 0 0.7181397206658644 rpy=0 0 0
- joint Link4_Link4XLink0: origin xyz=0.7401006488352597 0.3726422215019433 0 rpy=0 0 0 -> xyz=0.7002530986478599 0.30425698042340316 0 rpy=0 0 0
- joint Link4_Link4ZLink0: origin xyz=0 0.3726422215019433 0.6935533422687894 rpy=0 0 0 -> xyz=0 0.30425698042340316 0.6876660176680492 rpy=0 0 0
